File: TestV3_2020/TestV3.brd (EAGLE design)
At the start: 160 x 100 mm, 106 parts, among them Q1 600mA/40V, Q2 600mA/40V, Q3 600mA/40V, Q4 600mA/40V, U2 MP2451, U3 10k, U4 INA169

Commit message: Finished TPS54331 Buck Converter Board Layout and Isolation Final Size ~2.2*2.2cm But I should probably add some test points and fix the silkscreen
Parts:
- removed 2C10, 2C7: 10nF, JH:C0603
- removed 2C11, 2C12: 47uF/6.3v, JH:C1210
- removed 2C5, 2C6: 4.7uF, JH:C0603
- removed 2C8: 22UF, JH:C1210
- removed 2C9: 0.1uF, JH:C0603
- removed C1: 1nF, JH:C0603
- removed C2: 47pF, JH:C0603
- removed D2: SS34, SparkFun-DiscreteSemi:SMA-DIODE
- removed L1: 6.8uH, JH:SWPA8040
- removed R13: 68.1k, JH:R0603
- removed R14: 332k, JH:R0603
- removed R15: 10k, JH:R0603
- removed R16: 3.24k, JH:R0603
- removed R17: 29.4k, JH:R0603
- added 4C1: 22UF, JH:C1210
- added 4C10: 47pF, JH:C0603
- added 4C11: 4.7nF, JH:C0603
- added 4C12: 39pF, JH:C0603
- added 4C5: 0.1uF, JH:C0603
- added 4C6, 4C7: 47uF, JH:C1210
- added 4C8: 10nF, JH:C0603
- added 4C9: 1nF, JH:C0603
- added 4D1: SS34, SparkFun-DiscreteSemi:SMA-DIODE
- added 4JP1, 4JP2: JUMPER-SMT_3_NO_SILK, SparkFun-Jumpers:SMT-JUMPER_3_NO_SILK
- added 4L1: 6.8uH, JH:SWPA8040
- added 4R1: 180k, JH:R0603
- added 4R2: 51k, JH:R0603
- added 4R3: 10k, JH:R0603
- added 4R4: 29.4k, JH:R0603
- added 4R5: 49.9k, JH:R0603
- added 4R6: 3.24k, JH:R0603
- added 4R7: 1.91k, JH:R0603
- added J2: (no value), SparkFun-Connectors:1X05_LOCK
- added J4: (no value), SparkFun-Connectors:1X03_LOCK
- moved U1 56.1 mm to (76.2, 16.5)
- moved 3D1 5.46 mm to (-45.1, -62.9)
Connections:
- removed net N$13: R15.1, R16.1, U1.5
- new net COMP: 4JP1.2, U1.6
- new net GND-ISO: 4C1.2, 4C10.2, 4C12.2, 4C6.2, 4C7.2, 4C8.2, 4D1.A, 4R2.1, 4R4.2, 4R5.2, 4R6.1, 4R7.1, J4.2, U1.7, U1.9, U1.P$1, U1.P$2, U1.P$3, U1.P$4, U1.P$5, U1.P$6
- new net N$52: 4C11.2, 4R5.1
- new net N$54: 4C11.1, 4C12.1, 4JP1.3
- new net N$57: 4JP2.1, 4R6.2
- new net N$58: 4JP2.3, 4R7.2
- new net VIN: 4C1.1, 4R1.2, J4.3, U1.2
- new net VOUT: 4C6.1, 4C7.1, 4L1.P2, 4R3.2, J4.1
- new net VSNS: 4JP2.2, 4R3.1, U1.5
- net 12V: no longer 2C5.1, 2C6.1, 2C7.1, 2C8.1, R14.2, U1.2
- net 3.3V: no longer 2C11.1, 2C12.1, L1.P2, R15.2
- net GND: no longer 2C10.2, 2C11.2, 2C12.2, 2C5.2, 2C6.2, 2C7.2, 2C8.2, C2.2, D2.A, R13.1, R16.2, R17.2, U1.7, U1.9, U1.P$1, U1.P$2, U1.P$3, U1.P$4, U1.P$5, U1.P$6
- net N$10: now also 4C5.2, 4D1.C, 4L1.P1; no longer 2C9.2, D2.C, L1.P1
- net N$11: now also 4R1.1, 4R2.2; no longer R13.2, R14.1
- net N$12: now also 4C9.2, 4R4.1; no longer C1.2, R17.1
- net N$15: now also 4C10.1, 4C9.1, 4JP1.1; no longer C1.1, C2.1, U1.6
- net N$45: now also J2.5
- net N$46: now also J2.4
- net N$47: now also J2.3
- net N$48: now also J2.2
- net N$49: now also J2.1
- net N$8: now also 4C8.1; no longer 2C10.1
- net N$9: now also 4C5.1; no longer 2C9.1
Routing:
- net VIN: track 0.00 -> 24.7 mm, vias 0 -> 1
- net N$54: track 0.00 -> 17.4 mm, vias 0 -> 2
- net VSNS: track 0.00 -> 15.6 mm, vias 0 -> 1
- net N$8: track 0.00 -> 11.1 mm
- net N$11: track 0.00 -> 10.1 mm
- net N$15: track 0.00 -> 8.66 mm
- net N$58: track 0.00 -> 5.00 mm
- net N$57: track 0.00 -> 4.83 mm
- net VOUT: track 0.00 -> 4.62 mm, vias 0 -> 1
- net N$52: track 0.00 -> 4.54 mm
- net COMP: track 0.00 -> 4.12 mm, vias 0 -> 1
- net N$10: track 0.00 -> 3.59 mm, vias 0 -> 1
- net N$9: track 0.00 -> 3.23 mm, vias 0 -> 1
- net GND-ISO: track 0.00 -> 2.73 mm, vias 0 -> 4
- net N$12: track 0.00 -> 2.35 mm
- added copper zone on layer 1, net GND-ISO
- added copper zone on layer 16, net GND-ISO
- added copper zone on layer 1, net N$10
- added copper zone on layer 1, net VOUT

Commit message: Added TCS3200 Datasheet and updated buck converter board layout fixed the silkscreen for buck converter and finalise design
Parts:
- removed 3C5: 0.1uF, JH:C0603
- removed C10, C11: 47pF, JH:C0603
- removed C12, C17, C18, C4, C5, C6, C7: 1uF, JH:C0603
- removed C19: 4.7uF, JH:C0603
- removed C8, C9: 20pF, JH:C0603
- removed D1: BLUE, SparkFun-LED:LED-0603
- removed D4, D5: SS34, SparkFun-DiscreteSemi:SMA-DIODE
- removed FB1, FB2: 30Ω/1.8A, SparkFun-Coils:0603
- removed J3: (no value), SparkFun-Connectors:USB-B-MICRO-SMD
- removed OSC: 8MHz, SparkFun-Clocks:CRYSTAL-SMD-5X3.2-2PAD
- removed POT2: 10k, JH:3296-TRIMPOT
- removed Q1, Q2: 600mA/40V, SparkFun-DiscreteSemi:SOT23-3
- removed R1, R2, R4, R5: 1k, JH:R0603
- removed R10: 1.5k, JH:R0603
- removed R11: 36k, JH:R0603
- removed R12: 47k, JH:R0603
- removed R19: 0.15, SparkFun-Resistors:0805
- removed R20: 3k, JH:R0603
- removed R21, R3, R8, R9: 10k, JH:R0603
- removed R6, R7: 22, JH:R0603
- removed S1, S2: 34-MOMENTARY-SWITCH, JH:3*4-MOMENTARY-SWITCH
- removed U$6: LM393, JH:SOIC-8
- removed U4: INA169, SparkFun-IC-Special-Function:SOT23-5
- removed U6: (no value), SparkFun-IC-Power:SOT223
- removed UC1: STM32F103CBT6, JH:LQFP48
- added 1C1, 1C3, 1C6: 1uF, JH:C0603
- added 1C10, 1C9: 47pF, JH:C0603
- added 1C2, 1C4, 4C3: 10nF, JH:C0603
- added 1C5, 4C2: 4.7uF, JH:C0603
- added 1C7, 1C8: 20pF, JH:C0603
- added 1D1: BLUE, SparkFun-LED:LED-0603
- added 1FB1, 1FB2: 30Ω/1.8A, SparkFun-Coils:0603
- added 1J1: USB-MICROB, JH:USB-MICROB
- added 1J2, 1J3: (no value), SparkFun-Connectors:1X20_LOCK
- added 1OSC: 8MHz, SparkFun-Clocks:CRYSTAL-SMD-5X3.2-2PAD
- added 1Q1, 1Q2: 600mA/40V, SparkFun-DiscreteSemi:SOT23-3
- added 1R1, 1R2, 1R5, 1R6: 1k, JH:R0603
- added 1R10: 1.5k, JH:R0603
- added 1R11: 36k, JH:R0603
- added 1R12: 47k, JH:R0603
- added 1R3, 1R4, 1R9: 10k, JH:R0603
- added 1R7, 1R8: 22, JH:R0603
- added 1S1, 1S2: 34-MOMENTARY-SWITCH, JH:3*4-MOMENTARY-SWITCH
- added 1U1: STM32F103CBT6, JH:LQFP48
- added 1U2: (no value), SparkFun-IC-Power:SOT223
- added J10: (no value), SparkFun-Connectors:SCREWTERMINAL-5MM-3
- added J5: CONN_03, JH:1X03_LOCK
- added J6: XT30UPB-F, JH:XT30UPB-F
- added J7: (no value), SparkFun-Connectors:1X07_LOCK
- added J8: (no value), SparkFun-Connectors:SCREWTERMINAL-5MM-2
- added J9: (no value), SparkFun-Connectors:1X02_LOCK
- added R13: 20k, JH:R0603
- 4C1: value 22UF -> 22uF
- 4C6, 4C7: device JH:C1210 -> JH:C1206
- 4D1, D3: device SparkFun-DiscreteSemi:SMA-DIODE -> JH:SMA-DIODE
- 4JP1, 4JP2: value JUMPER-SMT_3_NO_SILK -> JUMPER-SMT_3_NO_NO-SILK; device SparkFun-Jumpers:SMT-JUMPER_3_NO_SILK -> SparkFun-Jumpers:SMT-JUMPER_3_NO_NO-SILK
- C13: value 2.2uF/6.3V -> 2.2uF
- C15, C16: value 10uF/16V -> 10uF
- J1: device SparkFun-Connectors:1X03_LOCK -> SparkFun-Connectors:1X07_LOCK
- J4: value (none) -> XT30UPB-F; device SparkFun-Connectors:1X03_LOCK -> JH:XT30UPB-F
- U3: value 10k -> (none)
- moved J4 366.3 mm to (-78.7, -299.7), turned to 0 degrees
- moved U3 264.9 mm to (-89.5, -336.6)
- moved J1 188.1 mm to (-83.2, -332.1)
- moved 2C1 164.6 mm to (-73.0, -125.7)
- moved 2C2 164.6 mm to (-76.8, -125.7)
- moved 2C3 164.6 mm to (-80.6, -125.7)
- moved 2C4 164.6 mm to (-84.5, -125.7)
- moved 2L1 164.6 mm to (-55.2, -125.7)
- moved 2R1 164.6 mm to (-69.2, -121.9)
- moved 2R2 164.6 mm to (-73.0, -121.9)
- moved 2R3 164.6 mm to (-76.8, -121.9)
- moved U2 164.6 mm to (-67.9, -125.7)
- moved D3 159.7 mm to (-61.6, -125.7)
- moved 3C3 143.4 mm to (-83.2, -198.1)
- moved SWD 136.5 mm to (-37.5, 133.3)
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Connections:
- removed net 12V: 2C1.1, 3C1.+, 3C5.1, 3L1.1, 3U1.P5, C19.1, D4.C, R23.2, R24.2, R25.1, U2.P5, U4.5, U6.3
- removed net 3.3V: 2C2.1, 2C3.1, 2L1.P2, 2R1.2, 2R3.1, 3C3.1, C12.1, C20.2, CS1.5, POT2.1, R20.2, U$6.8, U3.8
- removed net N$14: 3C4.+, 3D1.C, C3.+, R18.2, R19.1, U4.3
- removed net N$17: R21.2, U$6.3, U4.1
- removed net N$19: D5.A, R20.1, U$6.1
- removed net N$20: POT2.2, U$6.2
- removed net VCC_1: C14.2, C15.1, C16.1, R28.2, R29.2, U5.12
- removed net VCC_2: R19.2, U4.4
- new net GND-BOOST: 3C1.-, 3C2.2, 3C4.-, 3R2.1, 3U1.P$1, 3U1.P$10, 3U1.P$11, 3U1.P$12, 3U1.P$13, 3U1.P$14, 3U1.P$15, 3U1.P$16, 3U1.P$17, 3U1.P$18, 3U1.P$19, 3U1.P$2, 3U1.P$20, 3U1.P$3, 3U1.P$4, 3U1.P$5, 3U1.P$6, 3U1.P$7, 3U1.P$8, 3U1.P$9, 3U1.P3, 3U1.TAB, C3.-, J10.2
- new net GND-BUCK: 2C1.2, 2C2.2, 2R2.1, D3.A, U2.P2
- new net GND-CS: C20.1, CS1.4, J1.1, R30.1
- new net GND-LED: J9.1, Q3.2, Q4.2, R22.1
- new net GND-MOTOR: C13.2, C15.2, C16.2, J8.1, R26.1, R27.1, U5.13, U5.PPAD
- new net GND-POT: 3C3.2, J2.1, U3.4
- new net N$13: 1C5.1, 1U2.3
- new net VCC-MOTOR: J7.1, R28.2, R29.2
- new net VIN-BOOST: 3C1.+, 3L1.1, 3U1.P5, J10.3
- new net VIN-BUCK: 2C1.1, U2.P5
- new net VIN-CS: C20.2, CS1.5, J1.2
- new net VIN-LED: J9.2, R23.2, R24.2, R25.1
- new net VIN-MOTOR: C14.2, C15.1, C16.1, J8.2, U5.12
- new net VIN-POT: 3C3.1, J2.2, U3.8
- new net VOUT-BOOST: 3C4.+, 3D1.C, C3.+, J10.1, R18.2
- new net VOUT-BUCK: 2C2.1, 2C3.1, 2L1.P2, 2R1.2, 2R3.1
- net 0: now also 1J2.2, 1U1.22; no longer UC1.22
- net 1: now also 1J2.3, 1U1.21; no longer UC1.21
- net 10: now also 1J2.12, 1U1.11; no longer UC1.11
- net 11: now also 1J2.13, 1U1.10; no longer UC1.10
- net 12: now also 1J2.15, 1U1.4; no longer UC1.4
- net 13: now also 1J2.16, 1U1.3; no longer UC1.3
- net 14: now also 1J2.17, 1U1.2; no longer UC1.2
- net 15: now also 1J3.4, 1U1.43; no longer UC1.43
- net 16: now also 1J3.5, 1U1.42; no longer UC1.42
- net 17: now also 1J3.6, 1U1.41; no longer UC1.41
- net 18: now also 1J3.7, 1U1.40; no longer UC1.40
- net 19: now also 1J3.8, 1U1.39; no longer UC1.39
- net 2: now also 1J2.4, 1U1.20; no longer UC1.20
- net 20: now also 1J3.9, 1U1.38; no longer UC1.38
- net 21: now also 1J3.10, 1U1.37; no longer UC1.37
- net 22: now also 1J3.11, 1U1.34; no longer UC1.34
- net 23_USBDP: now also 1C10.2, 1J3.12, 1R10.1, 1R7.1, 1U1.33; no longer C11.2, R10.1, R7.1, UC1.33
- net 24_USBDM: now also 1C9.2, 1J3.13, 1R8.1, 1U1.32; no longer C10.2, R6.1, UC1.32
- net 25: now also 1J3.14, 1U1.31; no longer UC1.31
- net 26: now also 1J3.15, 1U1.30; no longer UC1.30
- net 27: now also 1J3.16, 1U1.29; no longer UC1.29
- net 28: now also 1J3.17, 1U1.28; no longer UC1.28
- net 29: now also 1J3.18, 1U1.27; no longer UC1.27
- net 3: now also 1J2.5, 1U1.18; no longer UC1.18
- net 30: now also 1J3.19, 1U1.26; no longer UC1.26
- net 31: now also 1J3.20, 1U1.25; no longer UC1.25
- net 32: now also 1J3.3, 1R3.2, 1S1.P2, 1U1.44, 1U1.45; no longer R9.2, S1.P2, UC1.44, UC1.45
- net 33: now also 1R1.2, 1U1.19; no longer R1.2, UC1.19
- net 4: now also 1J2.6, 1U1.17; no longer UC1.17
- net 5: now also 1J2.7, 1U1.16; no longer UC1.16
- net 6: now also 1J2.8, 1U1.15; no longer UC1.15
- net 7: now also 1J2.9, 1U1.14; no longer UC1.14
- net 8: now also 1J2.10, 1U1.13; no longer UC1.13
- net 9: now also 1J2.11, 1U1.12; no longer UC1.12
- net AGND: now also 1C1.2, 1C2.2, 1FB2.2, 1J2.19, 1U1.8; no longer C18.2, C4.2, FB2.2, UC1.8
- net DISC: now also 1R6.1, 1U1.46; no longer R5.1, UC1.46
- net FDBK: now also R13.1; no longer D5.C
- net GND: now also 1C10.1, 1C3.2, 1C4.2, 1C5.2, 1C6.2, 1C7.2, 1C8.2, 1C9.1, 1D1.C, 1FB2.1, 1J1.GND, 1J3.2, 1Q1.2, 1R11.1, 1R3.1, 1R5.1, 1U1.23, 1U1.35, 1U1.47, 1U2.1; no longer 2C1.2, 2C2.2, 2R2.1, 3C1.-, 3C2.2, 3C3.2, 3C4.-, 3C5.2, 3R2.1, 3U1.P$1, 3U1.P$10, 3U1.P$11, 3U1.P$12, 3U1.P$13, 3U1.P$14, 3U1.P$15, 3U1.P$16, 3U1.P$17, 3U1.P$18, 3U1.P$19, 3U1.P$2, 3U1.P$20, 3U1.P$3, 3U1.P$4, 3U1.P$5, 3U1.P$6, 3U1.P$7, 3U1.P$8, 3U1.P$9, 3U1.P3, 3U1.TAB, C10.1, C11.1, C12.2, C13.2, C15.2, C16.2, C17.2, C19.2, C20.1, C3.-, C5.2, C6.2, C7.2, C8.2, C9.2, CS1.4, D1.C, D3.A, FB2.1, J3.GND, POT2.3, Q1.2, Q3.2, Q4.2, R11.1, R21.1, R22.1, R26.1, R27.1, R30.1, R4.1, R9.1, U$6.4, U2.P2, U3.4, U4.2, U5.13, U5.PPAD, U6.1, UC1.23, UC1.35, UC1.47
- net GND-ISO: now also 4C2.2, 4C3.2, J5.2; no longer J4.2
- net N$1: now also 1R2.1, 1S1.P1; no longer R2.1, S1.P1
- net N$18: now also R13.2
- net N$2: now also 1D1.A, 1R1.1; no longer D1.A, R1.1
- net N$22: now also J2.3; no longer J1.1
- net N$23: now also J2.4; no longer J1.2
- net N$24: now also J2.5; no longer J1.3
- net N$27: now also J7.7
- net N$29: now also J7.6
- net N$30: now also J7.5
- net N$31: now also J7.4
- net N$32: now also J7.3
- net N$33: now also J7.2
- net N$39: now also J4.+
- net N$4: now also 1R5.2, 1S2.P1; no longer R4.2, S2.P1
- net N$40: now also J4.-
- net N$41: now also J6.+
- net N$42: now also J6.-
- net N$45: now also J1.7; no longer J2.5
- net N$46: now also J1.6; no longer J2.4
- net N$47: now also J1.5; no longer J2.3
- net N$48: now also J1.4; no longer J2.2
- net N$49: now also J1.3; no longer J2.1
- net N$51: now also 1Q2.2, 1R10.2; no longer Q2.2, R10.2
- net N$59: now also 1J1.D-, 1R8.2; no longer J3.D-, R6.2
- net N$60: now also 1J1.D+, 1R7.2; no longer J3.D+, R7.2
- net N$71: now also 1Q1.3, 1Q2.1, 1R11.2, 1R9.1; no longer Q1.3, Q2.1, R11.2, R8.1
- net N$73: now also 1Q1.1, 1R12.1, 1R6.2; no longer Q1.1, R12.1, R5.2
- net OSC_IN: now also 1C7.1, 1OSC.P$2, 1U1.5; no longer C9.1, OSC.P$2, UC1.5
- net OSC_OUT: now also 1C8.1, 1OSC.P$1, 1U1.6; no longer C8.1, OSC.P$1, UC1.6
- net RESET: now also 1J2.14, 1R4.1, 1S2.P2, 1U1.7; no longer R3.1, S2.P2, UC1.7
- net VBAT: now also 1J2.18, 1U1.1; no longer UC1.1
- net VCC: now also 1C3.1, 1C4.1, 1C6.1, 1FB1.1, 1J3.1, 1Q2.3, 1R12.2, 1R2.2, 1R4.2, 1U1.24, 1U1.36, 1U1.48, 1U2.2, 1U2.4; no longer C17.1, C5.1, C6.1, C7.1, FB1.1, Q2.3, R12.2, R2.2, R3.2, U6.2, U6.4, UC1.24, UC1.36, UC1.48
- net VCCA: now also 1C1.1, 1C2.1, 1FB1.2, 1J2.20, 1U1.9; no longer C18.1, C4.1, FB1.2, UC1.9
- net VIN: now also 4C2.1, 4C3.1, J5.3; no longer J4.3
- net VOUT: now also J5.1; no longer J4.1
- net V_USB: now also 1J1.VBUS, 1R9.2; no longer D4.A, J3.VBUS, R8.2
Routing:
- net VIN: track 24.7 -> 27.0 mm
- net VOUT: track 4.62 -> 3.98 mm
Other:
- board text added: "3.3v"
- board text added: "5v"
- board text added: "TPS54331 Buck Converter github.com/hcbozo"
- board text added: "WARNING: DO NOT power with jumpers unconnected MAX 5v out!!"
- board text added: "gnd"
- board text added: "vin"
- board text added: "vout"

Commit message: finished stm32 board layout, the end is near!
Parts:
- added 1C11: 1uF, JH:C0603
- 1C4: value 10nF -> 1uF
- moved J4 317.3 mm to (-31.1, 14.0)
- moved J9 317.3 mm to (-35.6, 33.7)
- moved C13 317.3 mm to (-24.8, -1.27)
- moved C14 317.3 mm to (-34.3, -1.27)
- moved C15 317.3 mm to (-32.4, -5.08)
- moved C16 317.3 mm to (-29.2, -5.08)
- moved C20 317.3 mm to (-35.6, -21.6)
- moved CS1 317.3 mm to (-33.7, -11.4)
- moved D6 317.3 mm to (-35.6, 26.7)
- moved J1 317.3 mm to (-35.6, -18.4)
- moved J10 317.3 mm to (-33.0, 45.1)
- moved J2 317.3 mm to (-35.6, 66.7)
- moved J6 317.3 mm to (-31.1, 7.62)
- moved J7 317.3 mm to (-35.6, 1.91)
- moved J8 317.3 mm to (-33.0, 20.3)
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Connections:
- net GND: now also 1C11.2
- net VCC: now also 1C11.1
Routing:
- net VCC: track 0.00 -> 138.2 mm, vias 0 -> 6
- net 23_USBDP: track 0.00 -> 30.9 mm, vias 0 -> 2
- net VCCA: track 0.00 -> 30.5 mm, vias 0 -> 2
- net AGND: track 0.00 -> 29.2 mm, vias 0 -> 2
- net 24_USBDM: track 0.00 -> 26.6 mm
- net RESET: track 0.00 -> 25.2 mm
- net 32: track 0.00 -> 24.9 mm
- net 31: track 0.00 -> 21.9 mm
- net 0: track 0.00 -> 20.3 mm
- net 30: track 0.00 -> 19.7 mm
- net 1: track 0.00 -> 17.8 mm
- net 29: track 0.00 -> 17.2 mm
- net VBAT: track 0.00 -> 16.9 mm
- net OSC_IN: track 0.00 -> 16.7 mm, vias 0 -> 1
- net 2: track 0.00 -> 15.5 mm
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- added copper zone on layer 1, net GND
- added copper zone on layer 16, net GND
- added copper zone on layer 1, net N$71
Other:
- board size 160 x 100 mm -> 100 x 100 mm
