File: PCB2k20/Layer1.sch (EAGLE design)
At the start: 0 parts

Commit message: Layer 3 placement kinda done, routing to wait for layer 1 signals to be confirmed. also renamed some folders because windows explorer doesnt like the old name
Parts:
- added 2C1, 2C2, 2C3: 0.1uF, JH:CAPACITOR0603
- added 2C4, 2C5, 2C6: 1uF, JH:CAPACITOR0603
- added 2R1, 2R2, 2R3: 1k, JH:RESISTOR0603
- added 2R4, 2R5, 2R6: 3k, JH:RESISTOR0603
- added LC1, LC2, LC3, LC4, LC5, LC6: (no value), JH:CAPACITOR0603
- added LD1, LD10, LD11, LD12, LD13, LD14, LD15, LD16, LD17, LD18, LD19, LD2, LD20, LD21, LD22, LD23, LD24, LD25, LD26, LD27, LD28, LD29, LD3, LD30, LD31, LD32, LD33, LD34, LD35, LD36, LD37, LD38, LD39, LD4, LD40, LD41, LD42, LD43, LD44, LD45, LD46, LD47, LD48, LD5, LD6, LD7, LD8, LD9: 3528LED, JH:3528LED
- added LG_D1: (no value), SparkFun-LED:LED5MM
- added LG_R1: PHOTOCELLPTH, SparkFun-Sensors:PHOTOCELLPTH
- added LG_R2, LR1: (no value), JH:RESISTOR0603
- added LS1: (no value), SparkFun-Switches:SWITCH-SPDT-PTH-11.6X4.0MM-LOCK
- added MUX_L1, MUX_L2, MUX_L3: (no value), JH:CD74HC4067SSOP-24
- added Q1, Q10, Q11, Q12, Q13, Q14, Q15, Q16, Q17, Q18, Q19, Q2, Q20, Q21, Q22, Q23, Q24, Q25, Q26, Q27, Q28, Q29, Q3, Q30, Q31, Q32, Q33, Q34, Q35, Q36, Q37, Q38, Q39, Q4, Q40, Q41, Q42, Q43, Q44, Q45, Q46, Q47, Q48, Q5, Q6, Q7, Q8, Q9: LIGHT_SENSORALS, SparkFun-Sensors:LIGHT_SENSORALS
Connections:
- new net 3.3V: 2C1.1, 2C2.1, 2C3.1, LG_D1.A, LG_R1.P$2, LS1.P, MUX_L1.VCC, MUX_L2.VCC, MUX_L3.VCC
- new net AGND: 2C4.2, 2C5.2, 2C6.2, 2R4.1, 2R5.1, 2R6.1
- new net GND: 2C1.2, 2C2.2, 2C3.2, 2R1.1, 2R2.1, 2R3.1, LC1.2, LC2.2, LC3.2, LC4.2, LC5.2, LC6.2, LG_D1.C, LG_R2.1, LR1.2, MUX_L1.GND, MUX_L2.GND, MUX_L3.GND
- new net LG_SIG: LG_R1.P$1, LG_R2.2
- new net LS0: MUX_L1.S0, MUX_L2.S0, MUX_L3.S0
- new net LS1: MUX_L1.S1, MUX_L2.S1, MUX_L3.S1
- new net LS2: MUX_L1.S2, MUX_L2.S2, MUX_L3.S2
- new net LS3: MUX_L1.S3, MUX_L2.S3, MUX_L3.S3
- new net LSIG1: 2C4.1, 2R4.2, MUX_L1.COM
- new net LSIG2: 2C5.1, 2R5.2, MUX_L2.COM
- new net LSIG3: 2C6.1, 2R6.2, MUX_L3.COM
- new net LSWITCH: LC1.1, LC2.1, LC3.1, LC4.1, LC5.1, LC6.1, LD1.A, LD10.A, LD11.A, LD12.A, LD13.A, LD14.A, LD15.A, LD16.A, LD17.A, LD18.A, LD19.A, LD2.A, LD20.A, LD21.A, LD22.A, LD23.A, LD24.A, LD25.A, LD26.A, LD27.A, LD28.A, LD29.A, LD3.A, LD30.A, LD31.A, LD32.A, LD33.A, LD34.A, LD35.A, LD36.A, LD37.A, LD38.A, LD39.A, LD4.A, LD40.A, LD41.A, LD42.A, LD43.A, LD44.A, LD45.A, LD46.A, LD47.A, LD48.A, LD5.A, LD6.A, LD7.A, LD8.A, LD9.A, LS1.O
- new net N$1: MUX_L1.CHAN15, Q1.E1
- new net N$10: MUX_L1.CHAN6, Q10.E1
- new net N$2: MUX_L1.CHAN14, Q2.E1
- new net N$3: MUX_L1.CHAN13, Q3.E1
- new net N$4: MUX_L1.CHAN12, Q4.E1
- new net N$5: MUX_L1.CHAN11, Q5.E1
- new net N$51: MUX_L1.CHAN5, Q11.E1
- new net N$52: 2R1.2, MUX_L1.EN
- new net N$53: MUX_L1.CHAN4, Q12.E1
- new net N$54: MUX_L1.CHAN3, Q13.E1
- new net N$55: MUX_L1.CHAN2, Q14.E1
- new net N$56: MUX_L1.CHAN1, Q15.E1
- new net N$57: MUX_L1.CHAN0, Q16.E1
- new net N$58: MUX_L2.CHAN15, Q17.E1
- new net N$59: MUX_L2.CHAN14, Q18.E1
- new net N$6: MUX_L1.CHAN10, Q6.E1
- new net N$60: MUX_L2.CHAN13, Q19.E1
- new net N$61: MUX_L2.CHAN12, Q20.E1
- new net N$62: MUX_L2.CHAN11, Q21.E1
- new net N$63: MUX_L2.CHAN10, Q22.E1
- new net N$64: MUX_L2.CHAN9, Q23.E1
- new net N$65: MUX_L2.CHAN8, Q24.E1
- new net N$66: MUX_L2.CHAN7, Q25.E1
- new net N$67: MUX_L2.CHAN6, Q26.E1
- new net N$68: MUX_L2.CHAN5, Q27.E1
- new net N$69: LD1.C, LD10.C, LD11.C, LD12.C, LD13.C, LD14.C, LD15.C, LD16.C, LD17.C, LD18.C, LD19.C, LD2.C, LD20.C, LD21.C, LD22.C, LD23.C, LD24.C, LD25.C, LD26.C, LD27.C, LD28.C, LD29.C, LD3.C, LD30.C, LD31.C, LD32.C, LD33.C, LD34.C, LD35.C, LD36.C, LD37.C, LD38.C, LD39.C, LD4.C, LD40.C, LD41.C, LD42.C, LD43.C, LD44.C, LD45.C, LD46.C, LD47.C, LD48.C, LD5.C, LD6.C, LD7.C, LD8.C, LD9.C, LR1.1
- new net N$7: MUX_L1.CHAN9, Q7.E1
- new net N$70: MUX_L2.CHAN4, Q28.E1
- new net N$71: MUX_L2.CHAN3, Q29.E1
- new net N$72: MUX_L2.CHAN2, Q30.E1
- new net N$73: MUX_L2.CHAN1, Q31.E1
- new net N$74: MUX_L2.CHAN0, Q32.E1
- new net N$75: MUX_L3.CHAN15, Q33.E1
- new net N$76: MUX_L3.CHAN14, Q34.E1
- new net N$77: MUX_L3.CHAN13, Q35.E1
- new net N$78: MUX_L3.CHAN12, Q36.E1
- new net N$79: MUX_L3.CHAN11, Q37.E1
- new net N$8: MUX_L1.CHAN8, Q8.E1
- new net N$80: MUX_L3.CHAN10, Q38.E1
- new net N$81: MUX_L3.CHAN9, Q39.E1
- new net N$82: 2R2.2, MUX_L2.EN
- new net N$83: MUX_L3.CHAN8, Q40.E1
- new net N$84: MUX_L3.CHAN7, Q41.E1
- new net N$85: MUX_L3.CHAN6, Q42.E1
- new net N$86: MUX_L3.CHAN5, Q43.E1
- new net N$87: MUX_L3.CHAN4, Q44.E1
- new net N$88: MUX_L3.CHAN3, Q45.E1
- new net N$89: MUX_L3.CHAN2, Q46.E1
- new net N$9: MUX_L1.CHAN7, Q9.E1
- new net N$90: MUX_L3.CHAN1, Q47.E1
- new net N$91: MUX_L3.CHAN0, Q48.E1
- new net N$99: 2R3.2, MUX_L3.EN
- new net VCCA: Q1.C1, Q10.C1, Q11.C1, Q12.C1, Q13.C1, Q14.C1, Q15.C1, Q16.C1, Q17.C1, Q18.C1, Q19.C1, Q2.C1, Q20.C1, Q21.C1, Q22.C1, Q23.C1, Q24.C1, Q25.C1, Q26.C1, Q27.C1, Q28.C1, Q29.C1, Q3.C1, Q30.C1, Q31.C1, Q32.C1, Q33.C1, Q34.C1, Q35.C1, Q36.C1, Q37.C1, Q38.C1, Q39.C1, Q4.C1, Q40.C1, Q41.C1, Q42.C1, Q43.C1, Q44.C1, Q45.C1, Q46.C1, Q47.C1, Q48.C1, Q5.C1, Q6.C1, Q7.C1, Q8.C1, Q9.C1
Other:
- note added: "motor switch"
