File: PCB2k20/Layer1.sch (EAGLE design)
At the start: 122 parts, among them Q1 LIGHT_SENSORALS, Q10 LIGHT_SENSORALS, Q11 LIGHT_SENSORALS, Q12 LIGHT_SENSORALS, Q13 LIGHT_SENSORALS, Q14 LIGHT_SENSORALS, Q15 LIGHT_SENSORALS, Q16 LIGHT_SENSORALS, Q17 LIGHT_SENSORALS, Q18 LIGHT_SENSORALS, Q19 LIGHT_SENSORALS, Q2 LIGHT_SENSORALS, Q20 LIGHT_SENSORALS, Q21 LIGHT_SENSORALS, Q22 LIGHT_SENSORALS, Q23 LIGHT_SENSORALS, Q24 LIGHT_SENSORALS, Q25 LIGHT_SENSORALS, Q26 LIGHT_SENSORALS, Q27 LIGHT_SENSORALS, Q28 LIGHT_SENSORALS, Q29 LIGHT_SENSORALS, Q3 LIGHT_SENSORALS, Q30 LIGHT_SENSORALS, Q31 LIGHT_SENSORALS, Q32 LIGHT_SENSORALS, Q33 LIGHT_SENSORALS, Q34 LIGHT_SENSORALS, Q35 LIGHT_SENSORALS, Q36 LIGHT_SENSORALS, Q37 LIGHT_SENSORALS, Q38 LIGHT_SENSORALS, Q39 LIGHT_SENSORALS, Q4 LIGHT_SENSORALS, Q40 LIGHT_SENSORALS, Q41 LIGHT_SENSORALS, Q42 LIGHT_SENSORALS, Q43 LIGHT_SENSORALS, Q44 LIGHT_SENSORALS, Q45 LIGHT_SENSORALS, Q46 LIGHT_SENSORALS, Q47 LIGHT_SENSORALS, Q48 LIGHT_SENSORALS, Q5 LIGHT_SENSORALS, Q6 LIGHT_SENSORALS, Q7 LIGHT_SENSORALS, Q8 LIGHT_SENSORALS, Q9 LIGHT_SENSORALS

Commit message: continue on layer 1 schematic, just need to finish this asap and quickly start positioning
Parts:
- removed 2C6: 1uF, JH:CAPACITOR0603
- removed 2R3: 1k, JH:RESISTOR0603
- removed 2R4, 2R5, 2R6: 3k, JH:RESISTOR0603
- removed LC1, LC2, LC3, LC4, LC5, LC6: (no value), JH:CAPACITOR0603
- removed LD1, LD10, LD11, LD12, LD13, LD14, LD15, LD16, LD17, LD18, LD19, LD2, LD20, LD21, LD22, LD23, LD24, LD25, LD26, LD27, LD28, LD29, LD3, LD30, LD31, LD32, LD33, LD34, LD35, LD36, LD37, LD38, LD39, LD4, LD40, LD41, LD42, LD43, LD44, LD45, LD46, LD47, LD48, LD5, LD6, LD7, LD8, LD9: 3528LED, JH:3528LED
- removed LG_D1: (no value), SparkFun-LED:LED5MM
- removed LG_R1: PHOTOCELLPTH, SparkFun-Sensors:PHOTOCELLPTH
- removed LG_R2, LR1: (no value), JH:RESISTOR0603
- removed LS1: (no value), SparkFun-Switches:SWITCH-SPDT-PTH-11.6X4.0MM-LOCK
- removed MUX_L1, MUX_L2, MUX_L3: (no value), JH:CD74HC4067SSOP-24
- removed Q1, Q10, Q11, Q12, Q13, Q14, Q15, Q16, Q17, Q18, Q19, Q2, Q20, Q21, Q22, Q23, Q24, Q25, Q26, Q27, Q28, Q29, Q3, Q30, Q31, Q32, Q33, Q34, Q35, Q36, Q37, Q38, Q39, Q4, Q40, Q41, Q42, Q43, Q44, Q45, Q46, Q47, Q48, Q5, Q6, Q7, Q8, Q9: LIGHT_SENSORALS, SparkFun-Sensors:LIGHT_SENSORALS
- added 1C1, 1C2, 1C3, 1C4, 1C5, 1C6: (no value), JH:CAPACITOR0603
- added 1C10, 1C9: 20pF, JH:CAPACITOR0603
- added 1C11, 1C12, 1C7, 1C8, 3C2: 1uF, JH:CAPACITOR0603
- added 1D1, 1D10, 1D11, 1D12, 1D13, 1D14, 1D15, 1D16, 1D17, 1D18, 1D19, 1D2, 1D20, 1D21, 1D22, 1D23, 1D24, 1D25, 1D26, 1D27, 1D28, 1D29, 1D3, 1D30, 1D31, 1D32, 1D33, 1D34, 1D35, 1D36, 1D4, 1D5, 1D6, 1D7, 1D8, 1D9: 3528LED, JH:3528LED
- added 1D37: BLUE, SparkFun-LED:LED-BLUE0603
- added 1OSC: 8MHz, SparkFun-Clocks:CRYSTALSMD-5X3.2-2PAD
- added 1PT1, 1PT10, 1PT11, 1PT12, 1PT13, 1PT14, 1PT15, 1PT16, 1PT17, 1PT18, 1PT19, 1PT2, 1PT20, 1PT21, 1PT22, 1PT23, 1PT24, 1PT25, 1PT26, 1PT27, 1PT28, 1PT29, 1PT3, 1PT30, 1PT31, 1PT32, 1PT33, 1PT34, 1PT35, 1PT36, 1PT4, 1PT5, 1PT6, 1PT7, 1PT8, 1PT9: LIGHT_SENSORALS, SparkFun-Sensors:LIGHT_SENSORALS
- added 1R1: 15, JH:RESISTOR0603
- added 1R10, 1R8: 1k, JH:RESISTOR0603
- added 1R11, 1R9, 3R3: 10k, JH:RESISTOR0603
- added 1R2, 1R3, 1R4, 1R5, 1R6, 1R7: (no value), JH:RESISTOR0603
- added 1SW1: MOMENTARY_SWITCH_4X3, JH:MOMENTARY_SWITCH_4X3
- added 1U1, 1U2, 1U3: (no value), JH:CD74HC4067SSOP-24
- added 1U4: STM32F103CBT6, JH:STM32F103CBT6
- added 2D1: 3A/40V/500mV, SparkFun-DiscreteSemi:DIODE-SCHOTTKY-B340A
- added 2L1: SWPA8040/10uH, JH:INDUCTORSWPA8040
- added 2U1: TPS5430, JH:TPS5450
- added 3C1: 100uF, SparkFun-Capacitors:100UF-POLAR-25V-20%(ELEC)
- added 3C3: 100uF, SparkFun-Capacitors:100UF-POLAR-10X10.5-63V-20%
- added 3C5: 0.1uF, JH:CAPACITOR0603
- added 3D1: SS510, diode:SCHOTTKY-DIODESMD
- added 3L1: 56uH, JH:INDUCTORCDRH127
- added 3POT1: 10k, JH:3296-TRIMPOT
- added 3R1: 2.94k, JH:RESISTOR0603
- added 3R2: 1.5k, JH:RESISTOR0603
- added 3R4: 47k, JH:RESISTOR0603
- added 3U1: LM2587, JH:LM2587
- added C1M1, C1M2, C1M3, C1M4: 33nF, SparkFun-Capacitors:33NF-0603-50V-10%
- added C2M1, C2M2, C2M3, C2M4: 680uF, rcl:CPOL-USE3.5-8
- added C3M1, C3M2, C3M3, C3M4: 1.0uF, SparkFun-Capacitors:1.0UF-0603-16V-10%-X7R
- added CONN_M1, CONN_M2, CONN_M3, CONN_M4: XT30PB-F, JH:XT30PB-F
- added D1M1, D1M2, D1M3, D1M4: GREEN, SparkFun-LED:LED-GREEN0603
- added D2M1, D2M2, D2M3, D2M4: RED, SparkFun-LED:LED-RED0603
- added FB1, FB2: 30Ω/1.8A, SparkFun-Coils:FERRITE_BEAD-0603
- added LIGHT: (no value), SparkFun-Switches:SWITCH-SPDT-PTH-11.6X4.0MM-LOCK
- added MOUSE: (no value), SparkFun-Connectors:CONN_08LOCK
- added Q1M1, Q1M2, Q1M3, Q1M4: AOD482, SparkFun-DiscreteSemi:MOSFET-NCH-FDD8780
- added R1: 300k, JH:RESISTOR0603
- added R10M1, R10M2, R10M3, R10M4, R3M1, R3M2, R3M3, R3M4, R4M1, R4M2, R4M3, R4M4, R5M1, R5M2, R5M3, R5M4, R6M1, R6M2, R6M3, R6M4, R7M1, R7M2, R7M3, R7M4: 1k, SparkFun-Resistors:1KOHM-0603-1/10W-1%
- added R11M1, R11M2, R11M3, R11M4, R8M1, R8M2, R8M3, R8M4, R9M1, R9M2, R9M3, R9M4: 10k, SparkFun-Resistors:10KOHM-0603-1/10W-1%
- added R12M1, R12M2, R12M3, R12M4: 4.7k, SparkFun-Resistors:4.7KOHM-0603-1/10W-1%
- added R1M1, R1M2, R1M3, R1M4, R2M1, R2M2, R2M3, R2M4: 3.3k, SparkFun-Resistors:3.3KOHM-0603-1/10W-1%
- added R2: 100k, JH:RESISTOR0603
- added SWD: JST_04-V, JH:JST_04-V
- added U$4, U$5: 74LVC2G, JH:74LVC2G
- added U1M1, U1M2, U1M3, U1M4: VNH5019, JH:VNH5019
- added U3: (no value), JH:MCP41XXX
- 2C1: value 0.1uF -> 22.0uF; device JH:CAPACITOR0603 -> JH:CAPACITOR1210
- 2C2: value 0.1uF -> 4.7uF
- 2C3: value 0.1uF -> 10.0nF
- 2C4: value 1uF -> 220uF; device JH:CAPACITOR0603 -> rcl:CPOL-USD/7343-31R
- 2C5: value 1uF -> 0.1uF
- 2R1: value 1k -> 10k
- 2R2: value 1k -> 5.9k
Connections:
- removed net LG_SIG: LG_R1.P$1, LG_R2.2
- removed net LS0: MUX_L1.S0, MUX_L2.S0, MUX_L3.S0
- removed net LS1: MUX_L1.S1, MUX_L2.S1, MUX_L3.S1
- removed net LS2: MUX_L1.S2, MUX_L2.S2, MUX_L3.S2
- removed net LS3: MUX_L1.S3, MUX_L2.S3, MUX_L3.S3
- removed net LSIG1: 2C4.1, 2R4.2, MUX_L1.COM
- removed net LSIG2: 2C5.1, 2R5.2, MUX_L2.COM
- removed net LSIG3: 2C6.1, 2R6.2, MUX_L3.COM
- removed net LSWITCH: LC1.1, LC2.1, LC3.1, LC4.1, LC5.1, LC6.1, LD1.A, LD10.A, LD11.A, LD12.A, LD13.A, LD14.A, LD15.A, LD16.A, LD17.A, LD18.A, LD19.A, LD2.A, LD20.A, LD21.A, LD22.A, LD23.A, LD24.A, LD25.A, LD26.A, LD27.A, LD28.A, LD29.A, LD3.A, LD30.A, LD31.A, LD32.A, LD33.A, LD34.A, LD35.A, LD36.A, LD37.A, LD38.A, LD39.A, LD4.A, LD40.A, LD41.A, LD42.A, LD43.A, LD44.A, LD45.A, LD46.A, LD47.A, LD48.A, LD5.A, LD6.A, LD7.A, LD8.A, LD9.A, LS1.O
- removed net N$89: MUX_L3.CHAN2, Q46.E1
- new net 12V: 2C1.1, 2C2.1, 2U1.VIN, 3C1.+, 3L1.1, 3U1.VIN
- new net 33: 1R8.2, 1U4.PB1/ADC12_IN9/TIM3_CH4
- new net BATT_LVL: R1.1, R2.1
- new net CPM1: Q1M1.G, U1M1.CP
- new net CPM2: Q1M2.G, U1M2.CP
- new net CPM3: Q1M3.G, U1M3.CP
- new net CPM4: Q1M4.G, U1M4.CP
- new net CSDIS1: R9M1.1, U1M1.CS_DIS
- new net CSDIS2: R9M2.1, U1M2.CS_DIS
- new net CSDIS3: R9M3.1, U1M3.CS_DIS
- new net CSDIS4: R9M4.1, U1M4.CS_DIS
- new net CSM1: C1M1.2, R8M1.1
- new net CSM2: C1M2.2, R8M2.1
- new net CSM3: C1M3.2, R8M3.1
- new net CSM4: C1M4.2, R8M4.1
- new net ENAM1: R3M1.1
- new net ENAM2: R3M2.1
- new net ENAM3: R3M3.1
- new net ENAM4: R3M4.1
- new net ENBM1: R4M1.2
- new net ENBM2: R4M2.2
- new net ENBM3: R4M3.2
- new net ENBM4: R4M4.2
- new net FDBK: 3POT1.CCW, 3POT1.WIPER, 3R2.2, 3U1.FDBK
- new net INBM1: R6M1.2, U$4G$1.Y
- new net INBM2: R6M2.2, U$4G$2.Y
- new net INBM3: R6M3.2, U$5G$1.Y
- new net INBM4: R6M4.2, U$5G$2.Y
- new net INM1: R5M1.1, U$4G$1.A
- new net INM2: R5M2.1, U$4G$2.A
- new net INM3: R5M3.1, U$5G$1.A
- new net INM4: R5M4.1, U$5G$2.A
- new net LSOUT1: 1C2.1, 1R3.2, 1U1.COM
- new net LSOUT2: 1C4.1, 1R5.2, 1U2.COM
- new net LSOUT3: 1C6.1, 1R7.2, 1U3.COM
- new net MOUSE_MISO: 1U4.PA6/SPI1_MISO/ADC12_IN6/TIM3_CH1, MOUSE.7
- new net MOUSE_MOSI: 1U4.PA7/SPI1_MOSI/ADC12_IN7/TIM3_CH2, MOUSE.8
- new net MOUSE_MOT: MOUSE.4
- new net MOUSE_RST: MOUSE.3
- new net MOUSE_SCK: 1U4.PA5/SPI1_SCK/ADC12_IN5, MOUSE.6
- new net MOUSE_SS: 1U4.PA4/SPI1_NSS/USART2_CK/ADC12_IN4, MOUSE.5
- new net N$100: 1R11.1, 1U4.BOOT0
- new net N$101: 2C3.2, 2D1.C, 2L1.1, 2U1.PH
- new net N$102: 2R1.1, 2R2.2, 2U1.VSNS
- new net N$103: 2C3.1, 2U1.BOOT
- new net N$104: D1M1.C, D2M1.A, R12M1.1
- new net N$11: 1PT8.E1, 1U1.CHAN8
- new net N$12: 1PT9.E1, 1U1.CHAN7
- new net N$13: 1PT10.E1, 1U1.CHAN6
- new net N$14: 1PT11.E1, 1U1.CHAN5
- new net N$15: 1PT12.E1, 1U1.CHAN4
- new net N$16: 1PT13.E1, 1U1.CHAN3
- new net N$17: 1PT14.E1, 1U1.CHAN2
- new net N$18: 1PT15.E1, 1U1.CHAN1
- new net N$19: 1PT16.E1, 1U1.CHAN0
- new net N$20: 1R2.2, 1U1.EN
- new net N$21: 1PT17.E1, 1U2.CHAN15
- new net N$22: 1C2.2, 1R3.1
- new net N$23: 1PT18.E1, 1U2.CHAN14
- new net N$24: 1PT19.E1, 1U2.CHAN13
- new net N$25: 1PT20.E1, 1U2.CHAN12
- new net N$26: 1PT21.E1, 1U2.CHAN11
- new net N$27: 1PT22.E1, 1U2.CHAN10
- new net N$28: 1PT23.E1, 1U2.CHAN9
- new net N$29: 1PT24.E1, 1U2.CHAN8
- new net N$30: 1PT25.E1, 1U2.CHAN7
- new net N$31: 1PT26.E1, 1U2.CHAN6
- new net N$32: 1PT27.E1, 1U2.CHAN5
- new net N$33: 1PT28.E1, 1U2.CHAN4
- new net N$34: 1PT29.E1, 1U2.CHAN3
- new net N$35: 1PT30.E1, 1U2.CHAN2
- new net N$36: 1PT31.E1, 1U2.CHAN1
- new net N$37: 1PT32.E1, 1U2.CHAN0
- new net N$38: 1R4.2, 1U2.EN
- new net N$39: 1C4.2, 1R5.1
- new net N$40: 1PT33.E1, 1U3.CHAN15
- new net N$41: 1PT34.E1, 1U3.CHAN14
- new net N$42: 1PT35.E1, 1U3.CHAN13
- new net N$43: 1PT36.E1, 1U3.CHAN12
- new net N$44: 1U3.CHAN11
- new net N$45: 1U3.CHAN10
- new net N$46: 1U3.CHAN9
- new net N$47: 1U3.CHAN8
- new net N$48: 1U3.CHAN7
- new net N$49: 1U3.CHAN6
- new net N$50: 1U3.CHAN5
- new net N$92: 3C2.1, 3R1.1
- new net N$93: 3POT1.CW, 3R3.1, U3POT1.CCW, U3POT1.WIPER
- new net N$94: 3R3.2, 3R4.1, U3POT1.CW
- new net N$98: 1R10.2, 1SW1.1
- new net OSC_IN: 1C9.1, 1OSC.2, 1U4.PD0-OSC_IN
- new net OSC_OUT: 1C10.1, 1OSC.1, 1U4.PD1-OSC_OUT
- new net OUTAM1: CONN_M1.P$V+, D1M1.A, D2M1.C, U1M1.OUT_A
- new net OUTAM2: CONN_M2.P$V+, D1M2.A, D2M2.C, U1M2.OUT_A
- new net OUTAM3: CONN_M3.P$V+, D1M3.A, D2M3.C, U1M3.OUT_A
- new net OUTAM4: CONN_M4.P$V+, D1M4.A, D2M4.C, U1M4.OUT_A
- new net OUTBM1: CONN_M1.P$V-, R12M1.2, U1M1.OUT_B
- new net OUTBM2: CONN_M2.P$V-, R12M2.2, U1M2.OUT_B
- new net OUTBM3: CONN_M3.P$V-, R12M3.2, U1M3.OUT_B
- new net OUTBM4: CONN_M4.P$V-, R12M4.2, U1M4.OUT_B
- new net POT_MOSI: 1U4.PB15/SPI2_MOSI/TIM1_CH3N, U3U1.MOSI
- new net POT_SCK: 1U4.PB13/SPI2_SCK/USART3_CTS/TIM1_CH1N, U3U1.SCLK
- new net POT_SS: 1U4.PB12/SPI2_NSS/I2C2_SMBA/USART3_CK/TIM1_BKIN, U3U1.CS
- new net PWMM1: R11M1.2, R7M1.2
- new net PWMM2: R11M2.2, R7M2.2
- new net PWMM3: R11M3.2, R7M3.2
- new net PWMM4: R11M4.2, R7M4.2
- new net RESET: 1R9.1, 1SW1.2, 1U4.NRST
- new net RX: 1U4.PA10/USART1_RX/TIM1_CH3
- new net S0: 1U1.S0, 1U2.S0, 1U3.S0
- new net S1: 1U1.S1, 1U2.S1, 1U3.S1
- new net S2: 1U1.S2, 1U2.S2, 1U3.S2
- new net S3: 1U1.S3, 1U2.S3, 1U3.S3
- new net SWDCLK: 1U4.PA14/JTCK/SWCLK, SWD.2
- new net SWDIO: 1U4.PA13/JTMS/SWDIO, SWD.3
- new net TX: 1U4.PA9/USART1_TX/TIM1_CH2
- new net VCC_1: Q1M1.S, Q1M2.S, Q1M3.S, Q1M4.S, R1.2, U1M1.VBAT, U1M2.VBAT, U1M3.VBAT, U1M4.VBAT
- new net VCC_2: 3C3.+, 3D1.C, 3R4.2
- net 3.3V: now also 1C1.1, 1C11.1, 1C3.1, 1C5.1, 1C7.1, 1C8.1, 1PT1.C1, 1PT10.C1, 1PT11.C1, 1PT12.C1, 1PT13.C1, 1PT14.C1, 1PT15.C1, 1PT16.C1, 1PT17.C1, 1PT18.C1, 1PT19.C1, 1PT2.C1, 1PT20.C1, 1PT21.C1, 1PT22.C1, 1PT23.C1, 1PT24.C1, 1PT25.C1, 1PT26.C1, 1PT27.C1, 1PT28.C1, 1PT29.C1, 1PT3.C1, 1PT30.C1, 1PT31.C1, 1PT32.C1, 1PT33.C1, 1PT34.C1, 1PT35.C1, 1PT36.C1, 1PT4.C1, 1PT5.C1, 1PT6.C1, 1PT7.C1, 1PT8.C1, 1PT9.C1, 1R9.2, 1U1.VCC, 1U2.VCC, 1U3.VCC, 1U4.VDD_1, 1U4.VDD_2, 1U4.VDD_3, 2C4.+, 2C5.1, 2L1.2, 2R1.2, 3C5.1, FB2.2, LIGHT.P, MOUSE.1, R1M1.2, R1M2.2, R1M3.2, R1M4.2, R2M1.2, R2M2.2, R2M3.2, R2M4.2, SWD.4, U$4G$3.P$V+, U$5G$3.P$V+, U3U1.VCC; no longer 2C1.1, 2C2.1, 2C3.1, LG_D1.A, LG_R1.P$2, LS1.P, MUX_L1.VCC, MUX_L2.VCC, MUX_L3.VCC
- net AGND: now also 1C12.1, 1U4.VSS_A, FB1.1; no longer 2C4.2, 2C5.2, 2C6.2, 2R4.1, 2R5.1, 2R6.1
- net GND: now also 1C1.2, 1C10.2, 1C11.2, 1C3.2, 1C5.2, 1C7.2, 1C8.2, 1C9.2, 1D21.C, 1D37.C, 1R10.1, 1R11.2, 1R2.1, 1R4.1, 1R6.1, 1U1.GND, 1U2.GND, 1U3.GND, 1U4.VSS_1, 1U4.VSS_2, 1U4.VSS_3, 2C4.-, 2C5.2, 2D1.A, 2U1.GND, 3C1.-, 3C2.2, 3C3.-, 3C5.2, 3R2.1, 3U1.GND, C1M1.1, C1M2.1, C1M3.1, C1M4.1, C2M1.-, C2M2.-, C2M3.-, C2M4.-, C3M1.2, C3M2.2, C3M3.2, C3M4.2, FB1.2, MOUSE.2, R10M1.1, R10M2.1, R10M3.1, R10M4.1, R11M1.1, R11M2.1, R11M3.1, R11M4.1, R2.2, R9M1.2, R9M2.2, R9M3.2, R9M4.2, SWD.1, U$4G$3.P$V-, U$5G$3.P$V-, U1M1.GND, U1M2.GND, U1M3.GND, U1M4.GND, U3U1.GND; no longer 2C3.2, 2R1.1, 2R3.1, LC1.2, LC2.2, LC3.2, LC4.2, LC5.2, LC6.2, LG_D1.C, LG_R2.1, LR1.2, MUX_L1.GND, MUX_L2.GND, MUX_L3.GND
- net N$1: now also 1D1.A, 1D10.A, 1D11.A, 1D12.A, 1D13.A, 1D14.A, 1D15.A, 1D16.A, 1D17.A, 1D18.A, 1D19.A, 1D2.A, 1D20.A, 1D21.A, 1D22.A, 1D23.A, 1D24.A, 1D25.A, 1D26.A, 1D27.A, 1D28.A, 1D29.A, 1D3.A, 1D30.A, 1D31.A, 1D32.A, 1D33.A, 1D34.A, 1D35.A, 1D36.A, 1D4.A, 1D5.A, 1D6.A, 1D7.A, 1D8.A, 1D9.A, 1R1.1; no longer MUX_L1.CHAN15, Q1.E1
- net N$10: now also 1PT7.E1, 1U1.CHAN9; no longer MUX_L1.CHAN6, Q10.E1
- net N$2: now also 1D1.C, 1D10.C, 1D11.C, 1D12.C, 1D13.C, 1D14.C, 1D15.C, 1D16.C, 1D17.C, 1D18.C, 1D19.C, 1D2.C, 1D20.C, 1D22.C, 1D23.C, 1D24.C, 1D25.C, 1D26.C, 1D27.C, 1D28.C, 1D29.C, 1D3.C, 1D30.C, 1D31.C, 1D32.C, 1D33.C, 1D34.C, 1D35.C, 1D36.C, 1D4.C, 1D5.C, 1D6.C, 1D7.C, 1D8.C, 1D9.C; no longer MUX_L1.CHAN14, Q2.E1
- net N$3: now also 1R1.2, LIGHT.S; no longer MUX_L1.CHAN13, Q3.E1
- net N$4: now also 1PT1.E1, 1U1.CHAN15; no longer MUX_L1.CHAN12, Q4.E1
- net N$5: now also 1PT2.E1, 1U1.CHAN14; no longer MUX_L1.CHAN11, Q5.E1
- net N$51: now also 1U3.CHAN4; no longer MUX_L1.CHAN5, Q11.E1
- net N$52: now also 1U3.CHAN3; no longer 2R1.2, MUX_L1.EN
- net N$53: now also 1U3.CHAN2; no longer MUX_L1.CHAN4, Q12.E1
- net N$54: now also 1U3.CHAN1; no longer MUX_L1.CHAN3, Q13.E1
- net N$55: now also 1U3.CHAN0; no longer MUX_L1.CHAN2, Q14.E1
- net N$56: now also 1R6.2, 1U3.EN; no longer MUX_L1.CHAN1, Q15.E1
- net N$57: now also 1C6.2, 1R7.1; no longer MUX_L1.CHAN0, Q16.E1
- net N$58: now also C2M1.+, C3M1.1, Q1M1.D, U1M1.VCC; no longer MUX_L2.CHAN15, Q17.E1
- net N$59: now also R2M1.1, R3M1.2, U1M1.EN_A; no longer MUX_L2.CHAN14, Q18.E1
- net N$6: now also 1PT3.E1, 1U1.CHAN13; no longer MUX_L1.CHAN10, Q6.E1
- net N$60: now also R5M1.2, U1M1.IN_A; no longer MUX_L2.CHAN13, Q19.E1
- net N$61: now also R1M1.1, R4M1.1, U1M1.EN_B; no longer MUX_L2.CHAN12, Q20.E1
- net N$62: now also R6M1.1, U1M1.IN_B; no longer MUX_L2.CHAN11, Q21.E1
- net N$63: now also R10M1.2, R8M1.2, U1M1.CS; no longer MUX_L2.CHAN10, Q22.E1
- net N$64: now also R7M1.1, U1M1.PWM_IN; no longer MUX_L2.CHAN9, Q23.E1
- net N$65: now also D1M2.C, D2M2.A, R12M2.1; no longer MUX_L2.CHAN8, Q24.E1
- net N$66: now also C2M2.+, C3M2.1, Q1M2.D, U1M2.VCC; no longer MUX_L2.CHAN7, Q25.E1
- net N$67: now also R2M2.1, R3M2.2, U1M2.EN_A; no longer MUX_L2.CHAN6, Q26.E1
- net N$68: now also R5M2.2, U1M2.IN_A; no longer MUX_L2.CHAN5, Q27.E1
- net N$69: now also R1M2.1, R4M2.1, U1M2.EN_B; no longer LD1.C, LD10.C, LD11.C, LD12.C, LD13.C, LD14.C, LD15.C, LD16.C, LD17.C, LD18.C, LD19.C, LD2.C, LD20.C, LD21.C, LD22.C, LD23.C, LD24.C, LD25.C, LD26.C, LD27.C, LD28.C, LD29.C, LD3.C, LD30.C, LD31.C, LD32.C, LD33.C, LD34.C, LD35.C, LD36.C, LD37.C, LD38.C, LD39.C, LD4.C, LD40.C, LD41.C, LD42.C, LD43.C, LD44.C, LD45.C, LD46.C, LD47.C, LD48.C, LD5.C, LD6.C, LD7.C, LD8.C, LD9.C, LR1.1
- net N$7: now also 1PT4.E1, 1U1.CHAN12; no longer MUX_L1.CHAN9, Q7.E1
- net N$70: now also R6M2.1, U1M2.IN_B; no longer MUX_L2.CHAN4, Q28.E1
- net N$71: now also R10M2.2, R8M2.2, U1M2.CS; no longer MUX_L2.CHAN3, Q29.E1
- net N$72: now also R7M2.1, U1M2.PWM_IN; no longer MUX_L2.CHAN2, Q30.E1
- net N$73: now also D1M3.C, D2M3.A, R12M3.1; no longer MUX_L2.CHAN1, Q31.E1
- net N$74: now also C2M3.+, C3M3.1, Q1M3.D, U1M3.VCC; no longer MUX_L2.CHAN0, Q32.E1
- net N$75: now also R2M3.1, R3M3.2, U1M3.EN_A; no longer MUX_L3.CHAN15, Q33.E1
- net N$76: now also R5M3.2, U1M3.IN_A; no longer MUX_L3.CHAN14, Q34.E1
- net N$77: now also R1M3.1, R4M3.1, U1M3.EN_B; no longer MUX_L3.CHAN13, Q35.E1
- net N$78: now also R6M3.1, U1M3.IN_B; no longer MUX_L3.CHAN12, Q36.E1
- net N$79: now also R10M3.2, R8M3.2, U1M3.CS; no longer MUX_L3.CHAN11, Q37.E1
- net N$8: now also 1PT5.E1, 1U1.CHAN11; no longer MUX_L1.CHAN8, Q8.E1
- net N$80: now also R7M3.1, U1M3.PWM_IN; no longer MUX_L3.CHAN10, Q38.E1
- net N$81: now also D1M4.C, D2M4.A, R12M4.1; no longer MUX_L3.CHAN9, Q39.E1
- net N$82: now also C2M4.+, C3M4.1, Q1M4.D, U1M4.VCC; no longer 2R2.2, MUX_L2.EN
- net N$83: now also R2M4.1, R3M4.2, U1M4.EN_A; no longer MUX_L3.CHAN8, Q40.E1
- net N$84: now also R5M4.2, U1M4.IN_A; no longer MUX_L3.CHAN7, Q41.E1
- net N$85: now also R1M4.1, R4M4.1, U1M4.EN_B; no longer MUX_L3.CHAN6, Q42.E1
- net N$86: now also R6M4.1, U1M4.IN_B; no longer MUX_L3.CHAN5, Q43.E1
- net N$87: now also R10M4.2, R8M4.2, U1M4.CS; no longer MUX_L3.CHAN4, Q44.E1
- net N$88: now also R7M4.1, U1M4.PWM_IN; no longer MUX_L3.CHAN3, Q45.E1
- net N$9: now also 1PT6.E1, 1U1.CHAN10; no longer MUX_L1.CHAN7, Q9.E1
- net N$90: now also 3D1.A, 3L1.2, 3U1.SW; no longer MUX_L3.CHAN1, Q47.E1
- net N$91: now also 3R1.2, 3U1.COMP; no longer MUX_L3.CHAN0, Q48.E1
- net N$99: now also 1D37.A, 1R8.1; no longer 2R3.2, MUX_L3.EN
- net VCCA: now also 1C12.2, 1U4.VDD_A, FB2.1; no longer Q1.C1, Q10.C1, Q11.C1, Q12.C1, Q13.C1, Q14.C1, Q15.C1, Q16.C1, Q17.C1, Q18.C1, Q19.C1, Q2.C1, Q20.C1, Q21.C1, Q22.C1, Q23.C1, Q24.C1, Q25.C1, Q26.C1, Q27.C1, Q28.C1, Q29.C1, Q3.C1, Q30.C1, Q31.C1, Q32.C1, Q33.C1, Q34.C1, Q35.C1, Q36.C1, Q37.C1, Q38.C1, Q39.C1, Q4.C1, Q40.C1, Q41.C1, Q42.C1, Q43.C1, Q44.C1, Q45.C1, Q46.C1, Q47.C1, Q48.C1, Q5.C1, Q6.C1, Q7.C1, Q8.C1, Q9.C1
Other:
- note added: "use xh2.54 here"

Commit message: placement done wow that was difficult
Parts:
- removed R3M1, R3M2, R3M3, R3M4, R4M1, R4M2, R4M3, R4M4: 1k, SparkFun-Resistors:1KOHM-0603-1/10W-1%
- added 1D0: BLUE, SparkFun-LED:LED-BLUE0603
- added 1D38, 1D39, 1D40: 3528LED, JH:3528LED
- added 1PT37, 1PT38, 1PT39, 1PT40, 1PT41, 1PT42: LIGHT_SENSORALS, SparkFun-Sensors:LIGHT_SENSORALS
- added 3C4: 1500uF, JH:1000UF-CAP
- added 3C7: 1500pF, JH:CAPACITOR0603
- added 3D4: 1N4728, diode:1N4728
- added 3D5: 1N5401, diode:1N5400
- added 3Q3: STP75NF75, SparkFun-DiscreteSemi:MOSFET-NCH-FQP30N06L
- added 3Q4: AO3400, SparkFun-DiscreteSemi:MOSFET-NCH-AO3404A
- added 3R10: 20, JH:RESISTOR0603
- added 3R7: 1k, JH:RESISTOR0603
- added 3R8, 3R9: 10k, JH:RESISTOR0603
- added C1, C2: 0.1uF, JH:CAPACITOR0603
- added GATE1, GATE2, THERM1, THERM2, THERM3, THERM4: (no value), SparkFun-Connectors:CONN_021X02_NO_SILK
- added J1: XT30PB-F, JH:XT30PB-F
- added R3, R4, R5, R6, R7, R8: (no value), JH:RESISTOR0603
- added S1: (no value), SparkFun-Switches:SWITCH-SPDT-PTH-11.6X4.0MM-LOCK
- 1D37: value BLUE -> 3528LED; device SparkFun-LED:LED-BLUE0603 -> JH:3528LED
- 3C1: device SparkFun-Capacitors:100UF-POLAR-25V-20%(ELEC) -> rcl:CPOL-USD
- 3R4: value 47k -> 47(+5)k
- C1M1, C1M2, C1M3, C1M4: device SparkFun-Capacitors:33NF-0603-50V-10% -> JH:CAPACITOR0603
- C3M1, C3M2, C3M3, C3M4: device SparkFun-Capacitors:1.0UF-0603-16V-10%-X7R -> JH:CAPACITOR0603
- R10M1, R10M2, R10M3, R10M4, R5M1, R5M2, R5M3, R5M4, R6M1, R6M2, R6M3, R6M4, R7M1, R7M2, R7M3, R7M4: device SparkFun-Resistors:1KOHM-0603-1/10W-1% -> JH:RESISTOR0603
- R11M1, R11M2, R11M3, R11M4: value 10k -> 100k; device SparkFun-Resistors:10KOHM-0603-1/10W-1% -> JH:RESISTOR0603
- R12M1, R12M2, R12M3, R12M4: device SparkFun-Resistors:4.7KOHM-0603-1/10W-1% -> JH:RESISTOR0603
- R1M1, R1M2, R1M3, R1M4, R2M1, R2M2, R2M3, R2M4: device SparkFun-Resistors:3.3KOHM-0603-1/10W-1% -> JH:RESISTOR0603
- R8M1, R8M2, R8M3, R8M4, R9M1, R9M2, R9M3, R9M4: device SparkFun-Resistors:10KOHM-0603-1/10W-1% -> JH:RESISTOR0603
- SWD: value JST_04-V -> BM06B-SRSS-TB; device JH:JST_04-V -> con-JST SH:BM06B-SRSS-TB
Connections:
- removed net ENAM1: R3M1.1
- removed net ENAM2: R3M2.1
- removed net ENAM3: R3M3.1
- removed net ENAM4: R3M4.1
- removed net ENBM1: R4M1.2
- removed net ENBM2: R4M2.2
- removed net ENBM3: R4M3.2
- removed net ENBM4: R4M4.2
- removed net N$2: 1D1.C, 1D10.C, 1D11.C, 1D12.C, 1D13.C, 1D14.C, 1D15.C, 1D16.C, 1D17.C, 1D18.C, 1D19.C, 1D2.C, 1D20.C, 1D22.C, 1D23.C, 1D24.C, 1D25.C, 1D26.C, 1D27.C, 1D28.C, 1D29.C, 1D3.C, 1D30.C, 1D31.C, 1D32.C, 1D33.C, 1D34.C, 1D35.C, 1D36.C, 1D4.C, 1D5.C, 1D6.C, 1D7.C, 1D8.C, 1D9.C
- removed net N$22: 1C2.2, 1R3.1
- removed net N$39: 1C4.2, 1R5.1
- removed net N$57: 1C6.2, 1R7.1
- new net 3.3V_MCU: 1C11.1, 1C7.1, 1C8.1, 1R9.2, 1U4.VDD_1, 1U4.VDD_2, 1U4.VDD_3, FB2.2, S1.P
- new net 3.3V_PROG: S1.S, SWD.4
- new net DEBUG_RX: 1U4.PA3/USART2_RX/ADC12_IN3/TIM2_CH4, SWD.6
- new net DEBUG_TX: 1U4.PA2/USART2_TX/ADC12_IN2/TIM2_CH3, SWD.5
- new net N$105: 3C7.1, 3R10.1
- new net N$106: GATE1.2, R3.2
- new net N$107: GATE2.2, R4.2
- new net N$95: 3C7.2, 3Q3.S, 3Q4.D, 3R8.1
- new net N$96: 3Q3.G, 3R7.2
- new net N$97: 3D4.C, 3D5.C
- new net SOLENOIDGND: 3D5.A, 3Q3.D, 3R10.2, J1.P$V-
- new net SOLENOIDON: 3Q4.G, 3R9.2
- net 12V: now also 3R7.1, 3R8.2; no longer 3C1.+, 3L1.1, 3U1.VIN
- net 3.3V: now also C1.1, C2.1, S1.O; no longer 1C1.1, 1C11.1, 1C3.1, 1C5.1, 1C7.1, 1C8.1, 1PT1.C1, 1PT10.C1, 1PT11.C1, 1PT12.C1, 1PT13.C1, 1PT14.C1, 1PT15.C1, 1PT16.C1, 1PT17.C1, 1PT18.C1, 1PT19.C1, 1PT2.C1, 1PT20.C1, 1PT21.C1, 1PT22.C1, 1PT23.C1, 1PT24.C1, 1PT25.C1, 1PT26.C1, 1PT27.C1, 1PT28.C1, 1PT29.C1, 1PT3.C1, 1PT30.C1, 1PT31.C1, 1PT32.C1, 1PT33.C1, 1PT34.C1, 1PT35.C1, 1PT36.C1, 1PT4.C1, 1PT5.C1, 1PT6.C1, 1PT7.C1, 1PT8.C1, 1PT9.C1, 1R9.2, 1U1.VCC, 1U2.VCC, 1U3.VCC, 1U4.VDD_1, 1U4.VDD_2, 1U4.VDD_3, FB2.2, SWD.4
- net AGND: now also 1C1.2, 1C2.2, 1C3.2, 1C4.2, 1C5.2, 1C6.2, 1R2.1, 1R3.1, 1R4.1, 1R5.1, 1R6.1, 1R7.1, 1U1.GND, 1U2.GND, 1U3.GND
- net GND: now also 1D0.C, 1D1.C, 1D10.C, 1D11.C, 1D12.C, 1D13.C, 1D14.C, 1D15.C, 1D16.C, 1D17.C, 1D18.C, 1D19.C, 1D2.C, 1D20.C, 1D22.C, 1D23.C, 1D24.C, 1D25.C, 1D26.C, 1D27.C, 1D28.C, 1D29.C, 1D3.C, 1D30.C, 1D31.C, 1D32.C, 1D33.C, 1D34.C, 1D35.C, 1D36.C, 1D38.C, 1D39.C, 1D4.C, 1D40.C, 1D5.C, 1D6.C, 1D7.C, 1D8.C, 1D9.C, 3C4.-, 3Q4.S, 3R9.1, C1.2, C2.2; no longer 1C1.2, 1C3.2, 1C5.2, 1R2.1, 1R4.1, 1R6.1, 1U1.GND, 1U2.GND, 1U3.GND
- net N$1: now also 1D37.A, 1D38.A, 1D39.A, 1D40.A
- net N$44: now also 1PT37.E1
- net N$45: now also 1PT38.E1
- net N$46: now also 1PT39.E1
- net N$47: now also 1PT40.E1
- net N$48: now also 1PT41.E1
- net N$49: now also 1PT42.E1
- net N$50: now also R5.1, THERM1.2
- net N$51: now also R6.1, THERM2.2
- net N$52: now also R7.1, THERM3.2
- net N$53: now also R8.1, THERM4.2
- net N$54: now also R3.1
- net N$55: now also R4.1
- net N$59: no longer R3M1.2
- net N$61: no longer R4M1.1
- net N$67: no longer R3M2.2
- net N$69: no longer R4M2.1
- net N$75: no longer R3M3.2
- net N$77: no longer R4M3.1
- net N$83: no longer R3M4.2
- net N$85: no longer R4M4.1
- net N$99: now also 1D0.A; no longer 1D37.A
- net VCCA: now also 1C1.1, 1C3.1, 1C5.1, 1PT1.C1, 1PT10.C1, 1PT11.C1, 1PT12.C1, 1PT13.C1, 1PT14.C1, 1PT15.C1, 1PT16.C1, 1PT17.C1, 1PT18.C1, 1PT19.C1, 1PT2.C1, 1PT20.C1, 1PT21.C1, 1PT22.C1, 1PT23.C1, 1PT24.C1, 1PT25.C1, 1PT26.C1, 1PT27.C1, 1PT28.C1, 1PT29.C1, 1PT3.C1, 1PT30.C1, 1PT31.C1, 1PT32.C1, 1PT33.C1, 1PT34.C1, 1PT35.C1, 1PT36.C1, 1PT37.C1, 1PT38.C1, 1PT39.C1, 1PT4.C1, 1PT40.C1, 1PT41.C1, 1PT42.C1, 1PT5.C1, 1PT6.C1, 1PT7.C1, 1PT8.C1, 1PT9.C1, 1U1.VCC, 1U2.VCC, 1U3.VCC, GATE1.1, GATE2.1, R5.2, R6.2, R7.2, R8.2, THERM1.1, THERM2.1, THERM3.1, THERM4.1
- net VCC_1: now also 3C1.+, 3L1.1, 3U1.VIN
- net VCC_2: now also 3C4.+, 3D4.A, J1.P$V+
Other:
- note added: "light interrupt"
- note removed: "use xh2.54 here"
- moved on the sheet: 1C10, 1C9, 1OSC, 2C1, 2C2, 2C3, 2C4, 2C5, 2D1, 2L1, 2R1, 2R2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

Commit message: half routed
Parts:
- added J2: CONN_03, JH:CONN_03
- added J3, J4, J5, U$16: 14AWG, JH:14AWG
- added LED1, LED2: (no value), SparkFun-Connectors:CONN_021X02_NO_SILK
- added U$15, U$17, U$18, U$19: 18AWG, JH:18AWG
- added X1: BM10B-SRSS-TB, con-JST SH:BM10B-SRSS-TB
Connections:
- new net LIGHT_INT: J2.1
- net 12V: now also U$15.1; no longer 3R7.1, 3R8.2
- net 3.3V: now also J2.3
- net GND: now also J2.2, LED1.2, LED2.2, U$18.1
- net INM1: now also X1.8
- net INM2: now also X1.6
- net INM3: now also X1.4
- net INM4: now also X1.2
- net MOUSE_MOT: now also 1U4.PB8/TIM4_CH3
- net MOUSE_RST: now also 1U4.PB9/TIM4_CH4
- net N$1: now also LED1.1, LED2.1, U$17.1
- net PWMM1: now also X1.7
- net PWMM2: now also X1.5
- net PWMM3: now also X1.3
- net PWMM4: now also X1.1
- net RX: now also X1.9
- net TX: now also X1.10
- net VCCA: now also U$19.1
- net VCC_1: now also 3R7.1, 3R8.2, J3.1, J4.1, J5.1, U$16.1

Commit message: done just need to silkscreen now!!!
Parts:
- removed 1D37, 1D39: 3528LED, JH:3528LED
- removed 1PT39, 1PT40, 1PT41, 1PT42: LIGHT_SENSORALS, SparkFun-Sensors:LIGHT_SENSORALS
- removed 3C5: 0.1uF, JH:CAPACITOR0603
- removed 3R3: 10k, JH:RESISTOR0603
- removed U3: (no value), JH:MCP41XXX
- added 1C13, 1C14, 1C15, 1C16, 1C17: (no value), JH:CAPACITOR0603
- added 1R12, 1R13, 1R14, 1R15, 1R16: (no value), JH:RESISTOR0603
- added C3: 1uF, JH:CAPACITOR0603
- added J10, J11, J13, J14, J15, J16, J17, J18, J19, J20, J6, J7, J8, J9: 14AWG, JH:14AWG
- added J12: (no value), SparkFun-Connectors:CONN_01
- added U$21, U$22, U$23, U$24, U$25, U$27, U$28: 18AWG, JH:18AWG
- added U$26: XT60XT60PB-M, JH:XT60XT60PB-M
- 3R4: value 47(+5)k -> 57k
- J2: value CONN_03 -> (none); device JH:CONN_03 -> SparkFun-Connectors:CONN_04
Connections:
- removed net N$106: GATE1.2, R3.2
- removed net N$107: GATE2.2, R4.2
- removed net N$41: 1PT34.E1, 1U3.CHAN14
- removed net N$42: 1PT35.E1, 1U3.CHAN13
- removed net N$43: 1PT36.E1, 1U3.CHAN12
- removed net N$44: 1PT37.E1, 1U3.CHAN11
- removed net N$45: 1PT38.E1, 1U3.CHAN10
- removed net N$46: 1PT39.E1, 1U3.CHAN9
- removed net N$47: 1PT40.E1, 1U3.CHAN8
- removed net N$48: 1PT41.E1, 1U3.CHAN7
- removed net N$49: 1PT42.E1, 1U3.CHAN6
- removed net N$50: 1U3.CHAN5, R5.1, THERM1.2
- removed net N$51: 1U3.CHAN4, R6.1, THERM2.2
- removed net N$52: 1U3.CHAN3, R7.1, THERM3.2
- removed net N$53: 1U3.CHAN2, R8.1, THERM4.2
- removed net N$54: 1U3.CHAN1, R3.1
- removed net N$55: 1U3.CHAN0, R4.1
- removed net N$93: 3POT1.CW, 3R3.1, U3POT1.CCW, U3POT1.WIPER
- removed net N$94: 3R3.2, 3R4.1, U3POT1.CW
- removed net POT_MOSI: 1U4.PB15/SPI2_MOSI/TIM1_CH3N, U3U1.MOSI
- removed net POT_SCK: 1U4.PB13/SPI2_SCK/USART3_CTS/TIM1_CH1N, U3U1.SCLK
- removed net POT_SS: 1U4.PB12/SPI2_NSS/I2C2_SMBA/USART3_CK/TIM1_BKIN, U3U1.CS
- new net GATE1: 1U3.CHAN10, GATE1.2, R3.2
- new net GATE2: 1U3.CHAN0, GATE2.2, R4.2
- new net L3>L1: J7.1, U$21.1, U$26.P$V+
- new net M1+2: J5.1, Q1M1.S, Q1M2.S, U1M1.VBAT, U1M2.VBAT
- new net MOTOR_SW: J10.1, J11.1, J20.1, J8.1, J9.1, R1.2
- new net N$2: 1PT26.E1, 1U2.CHAN15
- new net N$22: 1PT8.E1, 1U1.CHAN13
- new net N$39: J3.1, Q1M4.S, U1M4.VBAT
- new net PT22: 1C6.1, 1PT22.E1, 1R7.2, 1U3.CHAN1
- new net PT23: 1C13.1, 1PT23.E1, 1R12.2, 1U3.CHAN2
- new net PT24: 1C14.1, 1PT24.E1, 1R13.2, 1U3.CHAN3
- new net PT25: 1C15.1, 1PT25.E1, 1R14.2, 1U3.CHAN4
- new net PT37: 1C16.1, 1PT37.E1, 1R15.2, 1U3.CHAN12
- new net PT38: 1C17.1, 1PT38.E1, 1R16.2, 1U3.CHAN5
- new net THERM1: 1U3.CHAN13, R5.2, THERM1.2
- new net THERM2: 1U3.CHAN15, R6.2, THERM2.2
- new net THERM3: 1U3.CHAN8, R7.2, THERM3.2
- new net THERM4: 1U3.CHAN9, R8.2, THERM4.2
- net 3.3V: now also J2.4, U$28.1; no longer 3C5.1, LIGHT.P, U3U1.VCC
- net AGND: now also 1C13.2, 1C14.2, 1C15.2, 1C16.2, 1C17.2, 1R12.1, 1R13.1, 1R14.1, 1R15.1, 1R16.1, R3.1, R4.1, R5.1, R6.1, R7.1, R8.1
- net BATT_LVL: now also 1U4.PC13-TAMPER-RTC
- net CSM1: now also 1U3.CHAN11
- net CSM2: now also 1U3.CHAN14
- net CSM3: now also 1U3.CHAN7
- net CSM4: now also 1U3.CHAN6
- net GND: now also C3.2, J12.1, J13.1, J14.1, J15.1, J16.1, J17.1, J18.1, J19.1, J6.1, U$23.1, U$25.1, U$26.P$V-; no longer 1D37.C, 1D39.C, 3C5.2, U3U1.GND
- net LIGHT_INT: now also 1U4.PA11/USART1_CTS/CAN_RX/TIM1_CH4/USBDM
- net LSOUT1: now also 1U4.PB0/ADC12_IN8/TIM3_CH3
- net LSOUT2: now also 1U4.PA1/USART2_RTS/ADC12_IN1/TIM2_CH2
- net LSOUT3: now also 1U4.PA0_WKUP/USART2_CTS/ADC12_IN0/TIM2_CH1_ETR; no longer 1C6.1, 1R7.2
- net N$1: now also C3.1, U$22.1; no longer 1D37.A, 1D39.A
- net N$10: now also 1PT33.E1, 1U2.CHAN8; no longer 1PT7.E1, 1U1.CHAN9
- net N$11: now also 1PT34.E1, 1U2.CHAN7; no longer 1PT8.E1, 1U1.CHAN8
- net N$12: now also 1PT35.E1, 1U2.CHAN6; no longer 1PT9.E1, 1U1.CHAN7
- net N$13: now also 1PT36.E1, 1U2.CHAN5; no longer 1PT10.E1, 1U1.CHAN6
- net N$14: now also 1PT1.E1, 1U2.CHAN4; no longer 1PT11.E1, 1U1.CHAN5
- net N$15: now also 1PT2.E1, 1U2.CHAN3; no longer 1PT12.E1, 1U1.CHAN4
- net N$16: now also 1PT3.E1, 1U2.CHAN2; no longer 1PT13.E1, 1U1.CHAN3
- net N$17: now also 1PT4.E1, 1U2.CHAN1; no longer 1PT14.E1, 1U1.CHAN2
- net N$18: now also 1PT5.E1, 1U2.CHAN0; no longer 1PT15.E1, 1U1.CHAN1
- net N$19: now also 1PT6.E1, 1U1.CHAN15; no longer 1PT16.E1, 1U1.CHAN0
- net N$21: now also 1PT7.E1, 1U1.CHAN14; no longer 1PT17.E1, 1U2.CHAN15
- net N$23: now also 1PT9.E1, 1U1.CHAN12; no longer 1PT18.E1, 1U2.CHAN14
- net N$24: now also 1PT10.E1, 1U1.CHAN11; no longer 1PT19.E1, 1U2.CHAN13
- net N$25: now also 1PT11.E1, 1U1.CHAN10; no longer 1PT20.E1, 1U2.CHAN12
- net N$26: now also 1PT12.E1, 1U1.CHAN9; no longer 1PT21.E1, 1U2.CHAN11
- net N$27: now also 1PT13.E1, 1U1.CHAN8; no longer 1PT22.E1, 1U2.CHAN10
- net N$28: now also 1PT14.E1, 1U1.CHAN7; no longer 1PT23.E1, 1U2.CHAN9
- net N$29: now also 1PT15.E1, 1U1.CHAN6; no longer 1PT24.E1, 1U2.CHAN8
- net N$30: now also 1PT16.E1, 1U1.CHAN5; no longer 1PT25.E1, 1U2.CHAN7
- net N$31: now also 1PT17.E1, 1U1.CHAN4; no longer 1PT26.E1, 1U2.CHAN6
- net N$32: now also 1PT18.E1, 1U1.CHAN3; no longer 1PT27.E1, 1U2.CHAN5
- net N$33: now also 1PT19.E1, 1U1.CHAN2; no longer 1PT28.E1, 1U2.CHAN4
- net N$34: now also 1PT20.E1, 1U1.CHAN1; no longer 1PT29.E1, 1U2.CHAN3
- net N$35: now also 1PT21.E1, 1U1.CHAN0; no longer 1PT30.E1, 1U2.CHAN2
- net N$36: now also LIGHT.P, U$27.1; no longer 1PT31.E1, 1U2.CHAN1
- net N$37: now also 3POT1.CW, 3R4.1; no longer 1PT32.E1, 1U2.CHAN0
- net N$4: now also 1PT27.E1, 1U2.CHAN14; no longer 1PT1.E1, 1U1.CHAN15
- net N$40: now also J4.1, Q1M3.S, U1M3.VBAT; no longer 1PT33.E1, 1U3.CHAN15
- net N$5: now also 1PT28.E1, 1U2.CHAN13; no longer 1PT2.E1, 1U1.CHAN14
- net N$6: now also 1PT29.E1, 1U2.CHAN12; no longer 1PT3.E1, 1U1.CHAN13
- net N$7: now also 1PT30.E1, 1U2.CHAN11; no longer 1PT4.E1, 1U1.CHAN12
- net N$8: now also 1PT31.E1, 1U2.CHAN10; no longer 1PT5.E1, 1U1.CHAN11
- net N$9: now also 1PT32.E1, 1U2.CHAN9; no longer 1PT6.E1, 1U1.CHAN10
- net S0: now also 1U4.PA15/JTDI
- net S1: now also 1U4.PB3/JTDO
- net S2: now also 1U4.PB4/NJTRST
- net S3: now also 1U4.PB5/I2C1_SMBA
- net SOLENOIDON: now also 1U4.PA8/USART1_CK/TIM1_CH1/MCO
- net VCCA: now also U$24.1; no longer 1PT39.C1, 1PT40.C1, 1PT41.C1, 1PT42.C1, R5.2, R6.2, R7.2, R8.2
- net VCC_1: no longer J3.1, J4.1, J5.1, Q1M1.S, Q1M2.S, Q1M3.S, Q1M4.S, R1.2, U1M1.VBAT, U1M2.VBAT, U1M3.VBAT, U1M4.VBAT
Other:
- note removed: "light interrupt"
- note removed: "motor switch"
