File: PCB2k20/Layer1.brd (EAGLE design)
At the start: 173.9 x 196 mm, 0 parts

Commit message: Layer 3 placement kinda done, routing to wait for layer 1 signals to be confirmed. also renamed some folders because windows explorer doesnt like the old name
Parts:
- added 2C1, 2C2, 2C3: 0.1uF, JH:C0603
- added 2C4, 2C5, 2C6: 1uF, JH:C0603
- added 2R1, 2R2, 2R3: 1k, JH:R0603
- added 2R4, 2R5, 2R6: 3k, JH:R0603
- added LC1, LC2, LC3, LC4, LC5, LC6: (no value), JH:C0603
- added LD1, LD10, LD11, LD12, LD13, LD14, LD15, LD16, LD17, LD18, LD19, LD2, LD20, LD21, LD22, LD23, LD24, LD25, LD26, LD27, LD28, LD29, LD3, LD30, LD31, LD32, LD33, LD34, LD35, LD36, LD37, LD38, LD39, LD4, LD40, LD41, LD42, LD43, LD44, LD45, LD46, LD47, LD48, LD5, LD6, LD7, LD8, LD9: 3528LED, JH:3528
- added LG_D1: (no value), SparkFun-LED:LED_5MM
- added LG_R1: PHOTOCELLPTH, SparkFun-Sensors:PHOTOCELL
- added LG_R2, LR1: (no value), JH:R0603
- added LS1: (no value), SparkFun-Switches:SWITCH_SPDT_PTH_11.6X4.0MM_LOCK
- added MUX_L1, MUX_L2, MUX_L3: (no value), JH:SSOP24
- added Q1, Q10, Q11, Q12, Q13, Q14, Q15, Q16, Q17, Q18, Q19, Q2, Q20, Q21, Q22, Q23, Q24, Q25, Q26, Q27, Q28, Q29, Q3, Q30, Q31, Q32, Q33, Q34, Q35, Q36, Q37, Q38, Q39, Q4, Q40, Q41, Q42, Q43, Q44, Q45, Q46, Q47, Q48, Q5, Q6, Q7, Q8, Q9: (no value), SparkFun-Sensors:ALS-PT19
Connections:
- new net 3.3V: 2C1.1, 2C2.1, 2C3.1, LG_D1.A, LG_R1.2, LS1.2, MUX_L1.24, MUX_L2.24, MUX_L3.24
- new net AGND: 2C4.2, 2C5.2, 2C6.2, 2R4.1, 2R5.1, 2R6.1
- new net GND: 2C1.2, 2C2.2, 2C3.2, 2R1.1, 2R2.1, 2R3.1, LC1.2, LC2.2, LC3.2, LC4.2, LC5.2, LC6.2, LG_D1.K, LG_R2.1, LR1.2, MUX_L1.12, MUX_L2.12, MUX_L3.12
- new net LG_SIG: LG_R1.1, LG_R2.2
- new net LS0: MUX_L1.10, MUX_L2.10, MUX_L3.10
- new net LS1: MUX_L1.11, MUX_L2.11, MUX_L3.11
- new net LS2: MUX_L1.14, MUX_L2.14, MUX_L3.14
- new net LS3: MUX_L1.13, MUX_L2.13, MUX_L3.13
- new net LSIG1: 2C4.1, 2R4.2, MUX_L1.1
- new net LSIG2: 2C5.1, 2R5.2, MUX_L2.1
- new net LSIG3: 2C6.1, 2R6.2, MUX_L3.1
- new net LSWITCH: LC1.1, LC2.1, LC3.1, LC4.1, LC5.1, LC6.1, LD1.A, LD10.A, LD11.A, LD12.A, LD13.A, LD14.A, LD15.A, LD16.A, LD17.A, LD18.A, LD19.A, LD2.A, LD20.A, LD21.A, LD22.A, LD23.A, LD24.A, LD25.A, LD26.A, LD27.A, LD28.A, LD29.A, LD3.A, LD30.A, LD31.A, LD32.A, LD33.A, LD34.A, LD35.A, LD36.A, LD37.A, LD38.A, LD39.A, LD4.A, LD40.A, LD41.A, LD42.A, LD43.A, LD44.A, LD45.A, LD46.A, LD47.A, LD48.A, LD5.A, LD6.A, LD7.A, LD8.A, LD9.A, LS1.1
- new net N$1: MUX_L1.16, Q1.E
- new net N$10: MUX_L1.3, Q10.E
- new net N$2: MUX_L1.17, Q2.E
- new net N$3: MUX_L1.18, Q3.E
- new net N$4: MUX_L1.19, Q4.E
- new net N$5: MUX_L1.20, Q5.E
- new net N$51: MUX_L1.4, Q11.E
- new net N$52: 2R1.2, MUX_L1.15
- new net N$53: MUX_L1.5, Q12.E
- new net N$54: MUX_L1.6, Q13.E
- new net N$55: MUX_L1.7, Q14.E
- new net N$56: MUX_L1.8, Q15.E
- new net N$57: MUX_L1.9, Q16.E
- new net N$58: MUX_L2.16, Q17.E
- new net N$59: MUX_L2.17, Q18.E
- new net N$6: MUX_L1.21, Q6.E
- new net N$60: MUX_L2.18, Q19.E
- new net N$61: MUX_L2.19, Q20.E
- new net N$62: MUX_L2.20, Q21.E
- new net N$63: MUX_L2.21, Q22.E
- new net N$64: MUX_L2.22, Q23.E
- new net N$65: MUX_L2.23, Q24.E
- new net N$66: MUX_L2.2, Q25.E
- new net N$67: MUX_L2.3, Q26.E
- new net N$68: MUX_L2.4, Q27.E
- new net N$69: LD1.C, LD10.C, LD11.C, LD12.C, LD13.C, LD14.C, LD15.C, LD16.C, LD17.C, LD18.C, LD19.C, LD2.C, LD20.C, LD21.C, LD22.C, LD23.C, LD24.C, LD25.C, LD26.C, LD27.C, LD28.C, LD29.C, LD3.C, LD30.C, LD31.C, LD32.C, LD33.C, LD34.C, LD35.C, LD36.C, LD37.C, LD38.C, LD39.C, LD4.C, LD40.C, LD41.C, LD42.C, LD43.C, LD44.C, LD45.C, LD46.C, LD47.C, LD48.C, LD5.C, LD6.C, LD7.C, LD8.C, LD9.C, LR1.1
- new net N$7: MUX_L1.22, Q7.E
- new net N$70: MUX_L2.5, Q28.E
- new net N$71: MUX_L2.6, Q29.E
- new net N$72: MUX_L2.7, Q30.E
- new net N$73: MUX_L2.8, Q31.E
- new net N$74: MUX_L2.9, Q32.E
- new net N$75: MUX_L3.16, Q33.E
- new net N$76: MUX_L3.17, Q34.E
- new net N$77: MUX_L3.18, Q35.E
- new net N$78: MUX_L3.19, Q36.E
- new net N$79: MUX_L3.20, Q37.E
- new net N$8: MUX_L1.23, Q8.E
- new net N$80: MUX_L3.21, Q38.E
- new net N$81: MUX_L3.22, Q39.E
- new net N$82: 2R2.2, MUX_L2.15
- new net N$83: MUX_L3.23, Q40.E
- new net N$84: MUX_L3.2, Q41.E
- new net N$85: MUX_L3.3, Q42.E
- new net N$86: MUX_L3.4, Q43.E
- new net N$87: MUX_L3.5, Q44.E
- new net N$88: MUX_L3.6, Q45.E
- new net N$89: MUX_L3.7, Q46.E
- new net N$9: MUX_L1.2, Q9.E
- new net N$90: MUX_L3.8, Q47.E
- new net N$91: MUX_L3.9, Q48.E
- new net N$99: 2R3.2, MUX_L3.15
- new net VCCA: Q1.C, Q10.C, Q11.C, Q12.C, Q13.C, Q14.C, Q15.C, Q16.C, Q17.C, Q18.C, Q19.C, Q2.C, Q20.C, Q21.C, Q22.C, Q23.C, Q24.C, Q25.C, Q26.C, Q27.C, Q28.C, Q29.C, Q3.C, Q30.C, Q31.C, Q32.C, Q33.C, Q34.C, Q35.C, Q36.C, Q37.C, Q38.C, Q39.C, Q4.C, Q40.C, Q41.C, Q42.C, Q43.C, Q44.C, Q45.C, Q46.C, Q47.C, Q48.C, Q5.C, Q6.C, Q7.C, Q8.C, Q9.C

Commit message: continue on layer 1 schematic, just need to finish this asap and quickly start positioning
Parts:
- removed 2C6: 1uF, JH:C0603
- removed 2R3: 1k, JH:R0603
- removed 2R4, 2R5, 2R6: 3k, JH:R0603
- removed LC1, LC2, LC3, LC4, LC5, LC6: (no value), JH:C0603
- removed LD37, LD38, LD39, LD40, LD41, LD42, LD43, LD44, LD45, LD46, LD47, LD48: 3528LED, JH:3528
- removed LG_D1: (no value), SparkFun-LED:LED_5MM
- removed LG_R1: PHOTOCELLPTH, SparkFun-Sensors:PHOTOCELL
- removed LG_R2, LR1: (no value), JH:R0603
- removed LS1: (no value), SparkFun-Switches:SWITCH_SPDT_PTH_11.6X4.0MM_LOCK
- removed MUX_L1, MUX_L2, MUX_L3: (no value), JH:SSOP24
- removed Q37, Q38, Q39, Q40, Q41, Q42, Q43, Q44, Q45, Q46, Q47, Q48: (no value), SparkFun-Sensors:ALS-PT19
- added 1C1, 1C2, 1C3, 1C4, 1C5, 1C6: (no value), JH:C0603
- added 1C10, 1C9: 20pF, JH:C0603
- added 1C11, 1C12, 1C7, 1C8, 3C2: 1uF, JH:C0603
- added 1D37: BLUE, SparkFun-LED:LED-0603
- added 1OSC: 8MHz, SparkFun-Clocks:CRYSTAL-SMD-5X3.2-2PAD
- added 1R1: 15, JH:R0603
- added 1R10, 1R8: 1k, JH:R0603
- added 1R11, 1R9, 3R3: 10k, JH:R0603
- added 1R2, 1R3, 1R4, 1R5, 1R6, 1R7: (no value), JH:R0603
- added 1SW1: MOMENTARY_SWITCH_4X3, JH:MOMENTARY_SWITCH_4X3
- added 1U1, 1U2, 1U3: (no value), JH:SSOP24
- added 1U4: STM32F103CBT6, JH:LQFP48
- added 2D1: 3A/40V/500mV, SparkFun-DiscreteSemi:SMA-DIODE
- added 2L1: SWPA8040/10uH, JH:SWPA8040
- added 2U1: TPS5430, JH:POWERPAD-SOIC-8
- added 3C1: 100uF, SparkFun-Capacitors:PANASONIC_D
- added 3C3: 100uF, SparkFun-Capacitors:NIC_10X10.5_CAP
- added 3C5: 0.1uF, JH:C0603
- added 3D1: SS510, diode:SMB
- added 3L1: 56uH, JH:CDRH127
- added 3POT1: 10k, JH:3296-TRIMPOT
- added 3R1: 2.94k, JH:R0603
- added 3R2: 1.5k, JH:R0603
- added 3R4: 47k, JH:R0603
- added 3U1: LM2587, JH:TO-263
- added C1M1, C1M2, C1M3, C1M4: 33nF, SparkFun-Capacitors:0603
- added C2M1, C2M2, C2M3, C2M4: 680uF, rcl:E3,5-8
- added C3M1, C3M2, C3M3, C3M4: 1.0uF, SparkFun-Capacitors:0603
- added CONN_M1, CONN_M2, CONN_M3, CONN_M4: XT30PB-F, JH:XT30PB-F
- added D1M1, D1M2, D1M3, D1M4: GREEN, SparkFun-LED:LED-0603
- added D2M1, D2M2, D2M3, D2M4: RED, SparkFun-LED:LED-0603
- added FB1, FB2: 30Ω/1.8A, SparkFun-Coils:0603
- added LIGHT: (no value), SparkFun-Switches:SWITCH_SPDT_PTH_11.6X4.0MM_LOCK
- added MOUSE: (no value), SparkFun-Connectors:1X08_LOCK
- added Q1M1, Q1M2, Q1M3, Q1M4: AOD482, SparkFun-DiscreteSemi:DPAK
- added R1: 300k, JH:R0603
- added R10M1, R10M2, R10M3, R10M4, R3M1, R3M2, R3M3, R3M4, R4M1, R4M2, R4M3, R4M4, R5M1, R5M2, R5M3, R5M4, R6M1, R6M2, R6M3, R6M4, R7M1, R7M2, R7M3, R7M4: 1k, SparkFun-Resistors:0603
- added R11M1, R11M2, R11M3, R11M4, R8M1, R8M2, R8M3, R8M4, R9M1, R9M2, R9M3, R9M4: 10k, SparkFun-Resistors:0603
- added R12M1, R12M2, R12M3, R12M4: 4.7k, SparkFun-Resistors:0603
- added R1M1, R1M2, R1M3, R1M4, R2M1, R2M2, R2M3, R2M4: 3.3k, SparkFun-Resistors:0603
- added R2: 100k, JH:R0603
- added SWD: JST_04-V, JH:JST_04-V
- added U$4, U$5: 74LVC2G, JH:SOT23-6
- added U1M1, U1M2, U1M3, U1M4: VNH5019, JH:POWERSO-30
- added U3: (no value), JH:SOIC-8
- 1PT1, 1PT10, 1PT11, 1PT12, 1PT13, 1PT14, 1PT15, 1PT16, 1PT17, 1PT18, 1PT19, 1PT2, 1PT20, 1PT21, 1PT22, 1PT23, 1PT24, 1PT25, 1PT26, 1PT27, 1PT28, 1PT29, 1PT3, 1PT30, 1PT31, 1PT32, 1PT33, 1PT34, 1PT35, 1PT36, 1PT4, 1PT5, 1PT6, 1PT7, 1PT8, 1PT9: value (none) -> LIGHT_SENSORALS
- 2C1: value 0.1uF -> 22.0uF; device JH:C0603 -> JH:C1210
- 2C2: value 0.1uF -> 4.7uF
- 2C3: value 0.1uF -> 10.0nF
- 2C4: value 1uF -> 220uF; device JH:C0603 -> rcl:D/7343-31R
- 2C5: value 1uF -> 0.1uF
- 2R1: value 1k -> 10k
- 2R2: value 1k -> 5.9k
- moved 2C3 551.5 mm to (-528.3, -462.3)
- moved 2C1 549.8 mm to (-533.4, -463.6)
- moved 2C2 544.7 mm to (-524.5, -462.3)
- moved 2R1 523.9 mm to (-534.7, -468.6)
- moved 2R2 523.9 mm to (-530.9, -468.6)
- moved 2C4 505.6 mm to (-532.1, -455.9)
- moved 2C5 501.9 mm to (-520.7, -462.3)
- renumbered LD1 to 1D1, LD10 to 1D10, LD11 to 1D11, LD12 to 1D12, LD13 to 1D13, LD14 to 1D14, LD15 to 1D15, LD16 to 1D16, LD17 to 1D17, LD18 to 1D18, LD19 to 1D19, LD2 to 1D2, LD20 to 1D20, LD21 to 1D21, LD22 to 1D22, LD23 to 1D23, LD24 to 1D24, LD25 to 1D25, LD26 to 1D26, LD27 to 1D27, LD28 to 1D28, LD29 to 1D29, LD3 to 1D3, LD30 to 1D30, LD31 to 1D31, LD32 to 1D32, LD33 to 1D33, LD34 to 1D34, LD35 to 1D35, LD36 to 1D36, LD4 to 1D4, LD5 to 1D5, LD6 to 1D6, LD7 to 1D7, LD8 to 1D8, LD9 to 1D9, Q1 to 1PT1, Q10 to 1PT10, Q11 to 1PT11, Q12 to 1PT12, Q13 to 1PT13, Q14 to 1PT14, Q15 to 1PT15, Q16 to 1PT16, Q17 to 1PT17, Q18 to 1PT18, Q19 to 1PT19, Q2 to 1PT2, Q20 to 1PT20, Q21 to 1PT21, Q22 to 1PT22, Q23 to 1PT23, Q24 to 1PT24, Q25 to 1PT25, Q26 to 1PT26, Q27 to 1PT27, Q28 to 1PT28, Q29 to 1PT29, Q3 to 1PT3, Q30 to 1PT30, Q31 to 1PT31, Q32 to 1PT32, Q33 to 1PT33, Q34 to 1PT34, Q35 to 1PT35, Q36 to 1PT36, Q4 to 1PT4, Q5 to 1PT5, Q6 to 1PT6, Q7 to 1PT7, Q8 to 1PT8, Q9 to 1PT9
Connections:
- removed net LG_SIG: LG_R1.1, LG_R2.2
- removed net LS0: MUX_L1.10, MUX_L2.10, MUX_L3.10
- removed net LS1: MUX_L1.11, MUX_L2.11, MUX_L3.11
- removed net LS2: MUX_L1.14, MUX_L2.14, MUX_L3.14
- removed net LS3: MUX_L1.13, MUX_L2.13, MUX_L3.13
- removed net LSIG1: 2C4.1, 2R4.2, MUX_L1.1
- removed net LSIG2: 2C5.1, 2R5.2, MUX_L2.1
- removed net LSIG3: 2C6.1, 2R6.2, MUX_L3.1
- removed net LSWITCH: 1D1.A, 1D10.A, 1D11.A, 1D12.A, 1D13.A, 1D14.A, 1D15.A, 1D16.A, 1D17.A, 1D18.A, 1D19.A, 1D2.A, 1D20.A, 1D21.A, 1D22.A, 1D23.A, 1D24.A, 1D25.A, 1D26.A, 1D27.A, 1D28.A, 1D29.A, 1D3.A, 1D30.A, 1D31.A, 1D32.A, 1D33.A, 1D34.A, 1D35.A, 1D36.A, 1D4.A, 1D5.A, 1D6.A, 1D7.A, 1D8.A, 1D9.A, LC1.1, LC2.1, LC3.1, LC4.1, LC5.1, LC6.1, LD37.A, LD38.A, LD39.A, LD40.A, LD41.A, LD42.A, LD43.A, LD44.A, LD45.A, LD46.A, LD47.A, LD48.A, LS1.1
- removed net N$89: MUX_L3.7, Q46.E
- new net 12V: 2C1.1, 2C2.1, 2U1.7, 3C1.+, 3L1.1, 3U1.P5
- new net 33: 1R8.2, 1U4.19
- new net BATT_LVL: R1.1, R2.1
- new net CPM1: Q1M1.1, U1M1.P11
- new net CPM2: Q1M2.1, U1M2.P11
- new net CPM3: Q1M3.1, U1M3.P11
- new net CPM4: Q1M4.1, U1M4.P11
- new net CSDIS1: R9M1.1, U1M1.P6
- new net CSDIS2: R9M2.1, U1M2.P6
- new net CSDIS3: R9M3.1, U1M3.P6
- new net CSDIS4: R9M4.1, U1M4.P6
- new net CSM1: C1M1.2, R8M1.1
- new net CSM2: C1M2.2, R8M2.1
- new net CSM3: C1M3.2, R8M3.1
- new net CSM4: C1M4.2, R8M4.1
- new net ENAM1: R3M1.1
- new net ENAM2: R3M2.1
- new net ENAM3: R3M3.1
- new net ENAM4: R3M4.1
- new net ENBM1: R4M1.2
- new net ENBM2: R4M2.2
- new net ENBM3: R4M3.2
- new net ENBM4: R4M4.2
- new net FDBK: 3POT1.1, 3POT1.2, 3R2.2, 3U1.P2
- new net INBM1: R6M1.2, U$4.6
- new net INBM2: R6M2.2, U$4.4
- new net INBM3: R6M3.2, U$5.6
- new net INBM4: R6M4.2, U$5.4
- new net INM1: R5M1.1, U$4.1
- new net INM2: R5M2.1, U$4.3
- new net INM3: R5M3.1, U$5.1
- new net INM4: R5M4.1, U$5.3
- new net LSOUT1: 1C2.1, 1R3.2, 1U1.1
- new net LSOUT2: 1C4.1, 1R5.2, 1U2.1
- new net LSOUT3: 1C6.1, 1R7.2, 1U3.1
- new net MOUSE_MISO: 1U4.16, MOUSE.7
- new net MOUSE_MOSI: 1U4.17, MOUSE.8
- new net MOUSE_MOT: MOUSE.4
- new net MOUSE_RST: MOUSE.3
- new net MOUSE_SCK: 1U4.15, MOUSE.6
- new net MOUSE_SS: 1U4.14, MOUSE.5
- new net N$100: 1R11.1, 1U4.44
- new net N$101: 2C3.2, 2D1.C, 2L1.P1, 2U1.8
- new net N$102: 2R1.1, 2R2.2, 2U1.4
- new net N$103: 2C3.1, 2U1.1
- new net N$104: D1M1.C, D2M1.A, R12M1.1
- new net N$11: 1PT8.E, 1U1.23
- new net N$12: 1PT9.E, 1U1.2
- new net N$13: 1PT10.E, 1U1.3
- new net N$14: 1PT11.E, 1U1.4
- new net N$15: 1PT12.E, 1U1.5
- new net N$16: 1PT13.E, 1U1.6
- new net N$17: 1PT14.E, 1U1.7
- new net N$18: 1PT15.E, 1U1.8
- new net N$19: 1PT16.E, 1U1.9
- new net N$20: 1R2.2, 1U1.15
- new net N$21: 1PT17.E, 1U2.16
- new net N$22: 1C2.2, 1R3.1
- new net N$23: 1PT18.E, 1U2.17
- new net N$24: 1PT19.E, 1U2.18
- new net N$25: 1PT20.E, 1U2.19
- new net N$26: 1PT21.E, 1U2.20
- new net N$27: 1PT22.E, 1U2.21
- new net N$28: 1PT23.E, 1U2.22
- new net N$29: 1PT24.E, 1U2.23
- new net N$30: 1PT25.E, 1U2.2
- new net N$31: 1PT26.E, 1U2.3
- new net N$32: 1PT27.E, 1U2.4
- new net N$33: 1PT28.E, 1U2.5
- new net N$34: 1PT29.E, 1U2.6
- new net N$35: 1PT30.E, 1U2.7
- new net N$36: 1PT31.E, 1U2.8
- new net N$37: 1PT32.E, 1U2.9
- new net N$38: 1R4.2, 1U2.15
- new net N$39: 1C4.2, 1R5.1
- new net N$40: 1PT33.E, 1U3.16
- new net N$41: 1PT34.E, 1U3.17
- new net N$42: 1PT35.E, 1U3.18
- new net N$43: 1PT36.E, 1U3.19
- new net N$44: 1U3.20
- new net N$45: 1U3.21
- new net N$46: 1U3.22
- new net N$47: 1U3.23
- new net N$48: 1U3.2
- new net N$49: 1U3.3
- new net N$50: 1U3.4
- new net N$92: 3C2.1, 3R1.1
- new net N$93: 3POT1.3, 3R3.1, U3.5, U3.6
- new net N$94: 3R3.2, 3R4.1, U3.7
- new net N$98: 1R10.2, 1SW1.P$1
- new net OSC_IN: 1C9.1, 1OSC.P$2, 1U4.5
- new net OSC_OUT: 1C10.1, 1OSC.P$1, 1U4.6
- new net OUTAM1: CONN_M1.+, D1M1.A, D2M1.C, U1M1.P1, U1M1.P25, U1M1.P30, U1M1.SLUG2
- new net OUTAM2: CONN_M2.+, D1M2.A, D2M2.C, U1M2.P1, U1M2.P25, U1M2.P30, U1M2.SLUG2
- new net OUTAM3: CONN_M3.+, D1M3.A, D2M3.C, U1M3.P1, U1M3.P25, U1M3.P30, U1M3.SLUG2
- new net OUTAM4: CONN_M4.+, D1M4.A, D2M4.C, U1M4.P1, U1M4.P25, U1M4.P30, U1M4.SLUG2
- new net OUTBM1: CONN_M1.-, R12M1.2, U1M1.P15, U1M1.P16, U1M1.P21, U1M1.SLUG3
- new net OUTBM2: CONN_M2.-, R12M2.2, U1M2.P15, U1M2.P16, U1M2.P21, U1M2.SLUG3
- new net OUTBM3: CONN_M3.-, R12M3.2, U1M3.P15, U1M3.P16, U1M3.P21, U1M3.SLUG3
- new net OUTBM4: CONN_M4.-, R12M4.2, U1M4.P15, U1M4.P16, U1M4.P21, U1M4.SLUG3
- new net POT_MOSI: 1U4.28, U3.3
- new net POT_SCK: 1U4.26, U3.2
- new net POT_SS: 1U4.25, U3.1
- new net PWMM1: R11M1.2, R7M1.2
- new net PWMM2: R11M2.2, R7M2.2
- new net PWMM3: R11M3.2, R7M3.2
- new net PWMM4: R11M4.2, R7M4.2
- new net RESET: 1R9.1, 1SW1.P$2, 1U4.7
- new net RX: 1U4.31
- new net S0: 1U1.10, 1U2.10, 1U3.10
- new net S1: 1U1.11, 1U2.11, 1U3.11
- new net S2: 1U1.14, 1U2.14, 1U3.14
- new net S3: 1U1.13, 1U2.13, 1U3.13
- new net SWDCLK: 1U4.37, SWD.2
- new net SWDIO: 1U4.34, SWD.3
- new net TX: 1U4.30
- new net VBAT: 1U4.1
- new net VCC_1: Q1M1.3, Q1M2.3, Q1M3.3, Q1M4.3, R1.2, U1M1.P12, U1M2.P12, U1M3.P12, U1M4.P12
- new net VCC_2: 3C3.+, 3D1.C, 3R4.2
- net 3.3V: now also 1C1.1, 1C11.1, 1C3.1, 1C5.1, 1C7.1, 1C8.1, 1PT1.C, 1PT10.C, 1PT11.C, 1PT12.C, 1PT13.C, 1PT14.C, 1PT15.C, 1PT16.C, 1PT17.C, 1PT18.C, 1PT19.C, 1PT2.C, 1PT20.C, 1PT21.C, 1PT22.C, 1PT23.C, 1PT24.C, 1PT25.C, 1PT26.C, 1PT27.C, 1PT28.C, 1PT29.C, 1PT3.C, 1PT30.C, 1PT31.C, 1PT32.C, 1PT33.C, 1PT34.C, 1PT35.C, 1PT36.C, 1PT4.C, 1PT5.C, 1PT6.C, 1PT7.C, 1PT8.C, 1PT9.C, 1R9.2, 1U1.24, 1U2.24, 1U3.24, 1U4.24, 1U4.36, 1U4.48, 2C4.+, 2C5.1, 2L1.P2, 2R1.2, 3C5.1, FB2.2, LIGHT.2, MOUSE.1, R1M1.2, R1M2.2, R1M3.2, R1M4.2, R2M1.2, R2M2.2, R2M3.2, R2M4.2, SWD.4, U$4.5, U$5.5, U3.8; no longer 2C1.1, 2C2.1, 2C3.1, LG_D1.A, LG_R1.2, LS1.2, MUX_L1.24, MUX_L2.24, MUX_L3.24
- net AGND: now also 1C12.1, 1U4.8, FB1.1; no longer 2C4.2, 2C5.2, 2C6.2, 2R4.1, 2R5.1, 2R6.1
- net GND: now also 1C1.2, 1C10.2, 1C11.2, 1C3.2, 1C5.2, 1C7.2, 1C8.2, 1C9.2, 1D21.C, 1D37.C, 1R10.1, 1R11.2, 1R2.1, 1R4.1, 1R6.1, 1U1.12, 1U2.12, 1U3.12, 1U4.23, 1U4.35, 1U4.47, 2C4.-, 2C5.2, 2D1.A, 2U1.6, 2U1.9, 2U1.P$1, 2U1.P$2, 2U1.P$3, 2U1.P$4, 2U1.P$5, 2U1.P$6, 3C1.-, 3C2.2, 3C3.-, 3C5.2, 3R2.1, 3U1.P$1, 3U1.P$10, 3U1.P$11, 3U1.P$12, 3U1.P$13, 3U1.P$14, 3U1.P$15, 3U1.P$16, 3U1.P$17, 3U1.P$18, 3U1.P$19, 3U1.P$2, 3U1.P$20, 3U1.P$3, 3U1.P$4, 3U1.P$5, 3U1.P$6, 3U1.P$7, 3U1.P$8, 3U1.P$9, 3U1.P3, 3U1.TAB, C1M1.1, C1M2.1, C1M3.1, C1M4.1, C2M1.-, C2M2.-, C2M3.-, C2M4.-, C3M1.2, C3M2.2, C3M3.2, C3M4.2, FB1.2, MOUSE.2, R10M1.1, R10M2.1, R10M3.1, R10M4.1, R11M1.1, R11M2.1, R11M3.1, R11M4.1, R2.2, R9M1.2, R9M2.2, R9M3.2, R9M4.2, SWD.1, U$4.2, U$5.2, U1M1.P18, U1M1.P19, U1M1.P20, U1M1.P26, U1M1.P27, U1M1.P28, U1M2.P18, U1M2.P19, U1M2.P20, U1M2.P26, U1M2.P27, U1M2.P28, U1M3.P18, U1M3.P19, U1M3.P20, U1M3.P26, U1M3.P27, U1M3.P28, U1M4.P18, U1M4.P19, U1M4.P20, U1M4.P26, U1M4.P27, U1M4.P28, U3.4; no longer 2C3.2, 2R1.1, 2R3.1, LC1.2, LC2.2, LC3.2, LC4.2, LC5.2, LC6.2, LG_D1.K, LG_R2.1, LR1.2, MUX_L1.12, MUX_L2.12, MUX_L3.12
- net N$1: now also 1D1.A, 1D10.A, 1D11.A, 1D12.A, 1D13.A, 1D14.A, 1D15.A, 1D16.A, 1D17.A, 1D18.A, 1D19.A, 1D2.A, 1D20.A, 1D21.A, 1D22.A, 1D23.A, 1D24.A, 1D25.A, 1D26.A, 1D27.A, 1D28.A, 1D29.A, 1D3.A, 1D30.A, 1D31.A, 1D32.A, 1D33.A, 1D34.A, 1D35.A, 1D36.A, 1D4.A, 1D5.A, 1D6.A, 1D7.A, 1D8.A, 1D9.A, 1R1.1; no longer 1PT1.E, MUX_L1.16
- net N$10: now also 1PT7.E, 1U1.22; no longer 1PT10.E, MUX_L1.3
- net N$2: now also 1D1.C, 1D10.C, 1D11.C, 1D12.C, 1D13.C, 1D14.C, 1D15.C, 1D16.C, 1D17.C, 1D18.C, 1D19.C, 1D2.C, 1D20.C, 1D22.C, 1D23.C, 1D24.C, 1D25.C, 1D26.C, 1D27.C, 1D28.C, 1D29.C, 1D3.C, 1D30.C, 1D31.C, 1D32.C, 1D33.C, 1D34.C, 1D35.C, 1D36.C, 1D4.C, 1D5.C, 1D6.C, 1D7.C, 1D8.C, 1D9.C; no longer 1PT2.E, MUX_L1.17
- net N$3: now also 1R1.2, LIGHT.3; no longer 1PT3.E, MUX_L1.18
- net N$4: now also 1PT1.E, 1U1.16; no longer 1PT4.E, MUX_L1.19
- net N$5: now also 1PT2.E, 1U1.17; no longer 1PT5.E, MUX_L1.20
- net N$51: now also 1U3.5; no longer 1PT11.E, MUX_L1.4
- net N$52: now also 1U3.6; no longer 2R1.2, MUX_L1.15
- net N$53: now also 1U3.7; no longer 1PT12.E, MUX_L1.5
- net N$54: now also 1U3.8; no longer 1PT13.E, MUX_L1.6
- net N$55: now also 1U3.9; no longer 1PT14.E, MUX_L1.7
- net N$56: now also 1R6.2, 1U3.15; no longer 1PT15.E, MUX_L1.8
- net N$57: now also 1C6.2, 1R7.1; no longer 1PT16.E, MUX_L1.9
- net N$58: now also C2M1.+, C3M1.1, Q1M1.4, U1M1.P13, U1M1.P23, U1M1.P3, U1M1.SLUG1; no longer 1PT17.E, MUX_L2.16
- net N$59: now also R2M1.1, R3M1.2, U1M1.P5; no longer 1PT18.E, MUX_L2.17
- net N$6: now also 1PT3.E, 1U1.18; no longer 1PT6.E, MUX_L1.21
- net N$60: now also R5M1.2, U1M1.P4; no longer 1PT19.E, MUX_L2.18
- net N$61: now also R1M1.1, R4M1.1, U1M1.P9; no longer 1PT20.E, MUX_L2.19
- net N$62: now also R6M1.1, U1M1.P10; no longer 1PT21.E, MUX_L2.20
- net N$63: now also R10M1.2, R8M1.2, U1M1.P8; no longer 1PT22.E, MUX_L2.21
- net N$64: now also R7M1.1, U1M1.P7; no longer 1PT23.E, MUX_L2.22
- net N$65: now also D1M2.C, D2M2.A, R12M2.1; no longer 1PT24.E, MUX_L2.23
- net N$66: now also C2M2.+, C3M2.1, Q1M2.4, U1M2.P13, U1M2.P23, U1M2.P3, U1M2.SLUG1; no longer 1PT25.E, MUX_L2.2
- net N$67: now also R2M2.1, R3M2.2, U1M2.P5; no longer 1PT26.E, MUX_L2.3
- net N$68: now also R5M2.2, U1M2.P4; no longer 1PT27.E, MUX_L2.4
- net N$69: now also R1M2.1, R4M2.1, U1M2.P9; no longer 1D1.C, 1D10.C, 1D11.C, 1D12.C, 1D13.C, 1D14.C, 1D15.C, 1D16.C, 1D17.C, 1D18.C, 1D19.C, 1D2.C, 1D20.C, 1D21.C, 1D22.C, 1D23.C, 1D24.C, 1D25.C, 1D26.C, 1D27.C, 1D28.C, 1D29.C, 1D3.C, 1D30.C, 1D31.C, 1D32.C, 1D33.C, 1D34.C, 1D35.C, 1D36.C, 1D4.C, 1D5.C, 1D6.C, 1D7.C, 1D8.C, 1D9.C, LD37.C, LD38.C, LD39.C, LD40.C, LD41.C, LD42.C, LD43.C, LD44.C, LD45.C, LD46.C, LD47.C, LD48.C, LR1.1
- net N$7: now also 1PT4.E, 1U1.19; no longer 1PT7.E, MUX_L1.22
- net N$70: now also R6M2.1, U1M2.P10; no longer 1PT28.E, MUX_L2.5
- net N$71: now also R10M2.2, R8M2.2, U1M2.P8; no longer 1PT29.E, MUX_L2.6
- net N$72: now also R7M2.1, U1M2.P7; no longer 1PT30.E, MUX_L2.7
- net N$73: now also D1M3.C, D2M3.A, R12M3.1; no longer 1PT31.E, MUX_L2.8
- net N$74: now also C2M3.+, C3M3.1, Q1M3.4, U1M3.P13, U1M3.P23, U1M3.P3, U1M3.SLUG1; no longer 1PT32.E, MUX_L2.9
- net N$75: now also R2M3.1, R3M3.2, U1M3.P5; no longer 1PT33.E, MUX_L3.16
- net N$76: now also R5M3.2, U1M3.P4; no longer 1PT34.E, MUX_L3.17
- net N$77: now also R1M3.1, R4M3.1, U1M3.P9; no longer 1PT35.E, MUX_L3.18
- net N$78: now also R6M3.1, U1M3.P10; no longer 1PT36.E, MUX_L3.19
- net N$79: now also R10M3.2, R8M3.2, U1M3.P8; no longer MUX_L3.20, Q37.E
- net N$8: now also 1PT5.E, 1U1.20; no longer 1PT8.E, MUX_L1.23
- net N$80: now also R7M3.1, U1M3.P7; no longer MUX_L3.21, Q38.E
- net N$81: now also D1M4.C, D2M4.A, R12M4.1; no longer MUX_L3.22, Q39.E
- net N$82: now also C2M4.+, C3M4.1, Q1M4.4, U1M4.P13, U1M4.P23, U1M4.P3, U1M4.SLUG1; no longer 2R2.2, MUX_L2.15
- net N$83: now also R2M4.1, R3M4.2, U1M4.P5; no longer MUX_L3.23, Q40.E
- net N$84: now also R5M4.2, U1M4.P4; no longer MUX_L3.2, Q41.E
- net N$85: now also R1M4.1, R4M4.1, U1M4.P9; no longer MUX_L3.3, Q42.E
- net N$86: now also R6M4.1, U1M4.P10; no longer MUX_L3.4, Q43.E
- net N$87: now also R10M4.2, R8M4.2, U1M4.P8; no longer MUX_L3.5, Q44.E
- net N$88: now also R7M4.1, U1M4.P7; no longer MUX_L3.6, Q45.E
- net N$9: now also 1PT6.E, 1U1.21; no longer 1PT9.E, MUX_L1.2
- net N$90: now also 3D1.A, 3L1.2, 3U1.P4; no longer MUX_L3.8, Q47.E
- net N$91: now also 3R1.2, 3U1.P1; no longer MUX_L3.9, Q48.E
- net N$99: now also 1D37.A, 1R8.1; no longer 2R3.2, MUX_L3.15
- net VCCA: now also 1C12.2, 1U4.9, FB2.1; no longer 1PT1.C, 1PT10.C, 1PT11.C, 1PT12.C, 1PT13.C, 1PT14.C, 1PT15.C, 1PT16.C, 1PT17.C, 1PT18.C, 1PT19.C, 1PT2.C, 1PT20.C, 1PT21.C, 1PT22.C, 1PT23.C, 1PT24.C, 1PT25.C, 1PT26.C, 1PT27.C, 1PT28.C, 1PT29.C, 1PT3.C, 1PT30.C, 1PT31.C, 1PT32.C, 1PT33.C, 1PT34.C, 1PT35.C, 1PT36.C, 1PT4.C, 1PT5.C, 1PT6.C, 1PT7.C, 1PT8.C, 1PT9.C, Q37.C, Q38.C, Q39.C, Q40.C, Q41.C, Q42.C, Q43.C, Q44.C, Q45.C, Q46.C, Q47.C, Q48.C

Commit message: placement done wow that was difficult
Parts:
- removed R3M1, R3M2, R3M3, R3M4, R4M1, R4M2, R4M3, R4M4: 1k, SparkFun-Resistors:0603
- added 1D0: BLUE, SparkFun-LED:LED-0603
- added 1D38, 1D39, 1D40: 3528LED, JH:3528
- added 1PT37, 1PT38, 1PT39, 1PT40, 1PT41, 1PT42: LIGHT_SENSORALS, SparkFun-Sensors:ALS-PT19
- added 3C4: 1500uF, JH:1000UF-CAP
- added 3C7: 1500pF, JH:C0603
- added 3D4: 1N4728, diode:DO41Z10
- added 3D5: 1N5401, diode:DO201-15
- added 3Q3: STP75NF75, SparkFun-DiscreteSemi:TO220V
- added 3Q4: AO3400, SparkFun-DiscreteSemi:SOT23-3
- added 3R10: 20, JH:R0603
- added 3R7: 1k, JH:R0603
- added 3R8, 3R9: 10k, JH:R0603
- added C1, C2: 0.1uF, JH:C0603
- added GATE1, GATE2, THERM1, THERM2, THERM3, THERM4: (no value), SparkFun-Connectors:1X02_NO_SILK
- added J1: XT30PB-F, JH:XT30PB-F
- added R3, R4, R5, R6, R7, R8: (no value), JH:R0603
- added S1: (no value), SparkFun-Switches:SWITCH_SPDT_PTH_11.6X4.0MM_LOCK
- 1D37: value BLUE -> 3528LED; device SparkFun-LED:LED-0603 -> JH:3528
- 3C1: device SparkFun-Capacitors:PANASONIC_D -> rcl:PANASONIC_D
- 3R4: value 47k -> 47(+5)k
- C1M1, C1M2, C1M3, C1M4, C3M1, C3M2, C3M3, C3M4: device SparkFun-Capacitors:0603 -> JH:C0603
- R10M1, R10M2, R10M3, R10M4, R12M1, R12M2, R12M3, R12M4, R1M1, R1M2, R1M3, R1M4, R2M1, R2M2, R2M3, R2M4, R5M1, R5M2, R5M3, R5M4, R6M1, R6M2, R6M3, R6M4, R7M1, R7M2, R7M3, R7M4, R8M1, R8M2, R8M3, R8M4, R9M1, R9M2, R9M3, R9M4: device SparkFun-Resistors:0603 -> JH:R0603
- R11M1, R11M2, R11M3, R11M4: value 10k -> 100k; device SparkFun-Resistors:0603 -> JH:R0603
- SWD: value JST_04-V -> BM06B-SRSS-TB; device JH:JST_04-V -> con-JST SH:BM06B-SRSS-TB
- moved R12M2 815.5 mm to (36.2, 50.2), turned to 315 degrees
- moved D1M2 815.5 mm to (38.7, 51.4), turned to 225 degrees
- moved D2M2 812.7 mm to (37.5, 52.7), turned to 45 degrees
- moved CONN_M2 792.8 mm to (37.5, 24.8), turned to 225 degrees
- moved MOUSE 781.5 mm to (16.5, -16.5), turned to 90 degrees
- moved U$4 775.0 mm to (0.00, 52.1), turned to 90 degrees
- moved CONN_M3 768.3 mm to (37.5, -24.8), turned to 135 degrees
- moved R12M3 757.2 mm to (36.2, -50.2), turned to 225 degrees
- moved D1M3 753.6 mm to (37.5, -52.7), turned to 135 degrees
- moved D2M3 752.5 mm to (38.7, -51.4), turned to 315 degrees
- moved CONN_M1 740.9 mm to (-10.8, 51.4), turned to 315 degrees
- moved SWD 733.1 mm to (59.1, 25.4), turned to 270 degrees
- moved 1D37 732.6 mm to (0.00, 74.3), flipped to the bottom
- moved FB2 729.7 mm to (54.0, -6.99)
- moved R1 727.6 mm to (8.26, -79.4)
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Connections:
- removed net ENAM1: R3M1.1
- removed net ENAM2: R3M2.1
- removed net ENAM3: R3M3.1
- removed net ENAM4: R3M4.1
- removed net ENBM1: R4M1.2
- removed net ENBM2: R4M2.2
- removed net ENBM3: R4M3.2
- removed net ENBM4: R4M4.2
- removed net N$2: 1D1.C, 1D10.C, 1D11.C, 1D12.C, 1D13.C, 1D14.C, 1D15.C, 1D16.C, 1D17.C, 1D18.C, 1D19.C, 1D2.C, 1D20.C, 1D22.C, 1D23.C, 1D24.C, 1D25.C, 1D26.C, 1D27.C, 1D28.C, 1D29.C, 1D3.C, 1D30.C, 1D31.C, 1D32.C, 1D33.C, 1D34.C, 1D35.C, 1D36.C, 1D4.C, 1D5.C, 1D6.C, 1D7.C, 1D8.C, 1D9.C
- removed net N$22: 1C2.2, 1R3.1
- removed net N$39: 1C4.2, 1R5.1
- removed net N$57: 1C6.2, 1R7.1
- new net 3.3V_MCU: 1C11.1, 1C7.1, 1C8.1, 1R9.2, 1U4.24, 1U4.36, 1U4.48, FB2.2, S1.2
- new net 3.3V_PROG: S1.3, SWD.4
- new net DEBUG_RX: 1U4.13, SWD.6
- new net DEBUG_TX: 1U4.12, SWD.5
- new net N$105: 3C7.1, 3R10.1
- new net N$106: GATE1.2, R3.2
- new net N$107: GATE2.2, R4.2
- new net N$95: 3C7.2, 3Q3.3, 3Q4.3, 3R8.1
- new net N$96: 3Q3.1, 3R7.2
- new net N$97: 3D4.C, 3D5.C
- new net SOLENOIDGND: 3D5.A, 3Q3.2, 3R10.2, J1.-
- new net SOLENOIDON: 3Q4.1, 3R9.2
- net 12V: now also 3R7.1, 3R8.2; no longer 3C1.+, 3L1.1, 3U1.P5
- net 3.3V: now also C1.1, C2.1, S1.1; no longer 1C1.1, 1C11.1, 1C3.1, 1C5.1, 1C7.1, 1C8.1, 1PT1.C, 1PT10.C, 1PT11.C, 1PT12.C, 1PT13.C, 1PT14.C, 1PT15.C, 1PT16.C, 1PT17.C, 1PT18.C, 1PT19.C, 1PT2.C, 1PT20.C, 1PT21.C, 1PT22.C, 1PT23.C, 1PT24.C, 1PT25.C, 1PT26.C, 1PT27.C, 1PT28.C, 1PT29.C, 1PT3.C, 1PT30.C, 1PT31.C, 1PT32.C, 1PT33.C, 1PT34.C, 1PT35.C, 1PT36.C, 1PT4.C, 1PT5.C, 1PT6.C, 1PT7.C, 1PT8.C, 1PT9.C, 1R9.2, 1U1.24, 1U2.24, 1U3.24, 1U4.24, 1U4.36, 1U4.48, FB2.2, SWD.4
- net AGND: now also 1C1.2, 1C2.2, 1C3.2, 1C4.2, 1C5.2, 1C6.2, 1R2.1, 1R3.1, 1R4.1, 1R5.1, 1R6.1, 1R7.1, 1U1.12, 1U2.12, 1U3.12
- net GND: now also 1D0.C, 1D1.C, 1D10.C, 1D11.C, 1D12.C, 1D13.C, 1D14.C, 1D15.C, 1D16.C, 1D17.C, 1D18.C, 1D19.C, 1D2.C, 1D20.C, 1D22.C, 1D23.C, 1D24.C, 1D25.C, 1D26.C, 1D27.C, 1D28.C, 1D29.C, 1D3.C, 1D30.C, 1D31.C, 1D32.C, 1D33.C, 1D34.C, 1D35.C, 1D36.C, 1D38.C, 1D39.C, 1D4.C, 1D40.C, 1D5.C, 1D6.C, 1D7.C, 1D8.C, 1D9.C, 3C4.-, 3Q4.2, 3R9.1, C1.2, C2.2; no longer 1C1.2, 1C3.2, 1C5.2, 1R2.1, 1R4.1, 1R6.1, 1U1.12, 1U2.12, 1U3.12
- net N$1: now also 1D37.A, 1D38.A, 1D39.A, 1D40.A
- net N$44: now also 1PT37.E
- net N$45: now also 1PT38.E
- net N$46: now also 1PT39.E
- net N$47: now also 1PT40.E
- net N$48: now also 1PT41.E
- net N$49: now also 1PT42.E
- net N$50: now also R5.1, THERM1.2
- net N$51: now also R6.1, THERM2.2
- net N$52: now also R7.1, THERM3.2
- net N$53: now also R8.1, THERM4.2
- net N$54: now also R3.1
- net N$55: now also R4.1
- net N$59: no longer R3M1.2
- net N$61: no longer R4M1.1
- net N$67: no longer R3M2.2
- net N$69: no longer R4M2.1
- net N$75: no longer R3M3.2
- net N$77: no longer R4M3.1
- net N$83: no longer R3M4.2
- net N$85: no longer R4M4.1
- net N$99: now also 1D0.A; no longer 1D37.A
- net VCCA: now also 1C1.1, 1C3.1, 1C5.1, 1PT1.C, 1PT10.C, 1PT11.C, 1PT12.C, 1PT13.C, 1PT14.C, 1PT15.C, 1PT16.C, 1PT17.C, 1PT18.C, 1PT19.C, 1PT2.C, 1PT20.C, 1PT21.C, 1PT22.C, 1PT23.C, 1PT24.C, 1PT25.C, 1PT26.C, 1PT27.C, 1PT28.C, 1PT29.C, 1PT3.C, 1PT30.C, 1PT31.C, 1PT32.C, 1PT33.C, 1PT34.C, 1PT35.C, 1PT36.C, 1PT37.C, 1PT38.C, 1PT39.C, 1PT4.C, 1PT40.C, 1PT41.C, 1PT42.C, 1PT5.C, 1PT6.C, 1PT7.C, 1PT8.C, 1PT9.C, 1U1.24, 1U2.24, 1U3.24, GATE1.1, GATE2.1, R5.2, R6.2, R7.2, R8.2, THERM1.1, THERM2.1, THERM3.1, THERM4.1
- net VCC_1: now also 3C1.+, 3L1.1, 3U1.P5
- net VCC_2: now also 3C4.+, 3D4.A, J1.+
Other:
- outline, holes or cut-outs redrawn
