File: PCB2k20/Layer1.brd (EAGLE design)
At the start: 173.9 x 196 mm, 281 parts, among them J1 XT30PB-F, J10 14AWG, J11 14AWG, J13 14AWG, J14 14AWG, J15 14AWG, J16 14AWG, J17 14AWG, J18 14AWG, J19 14AWG, J20 14AWG, J21 14AWG, J3 14AWG, J4 14AWG, J5 14AWG, J6 14AWG, J7 14AWG, J8 14AWG, J9 14AWG, Q1M1 AOD482, Q1M2 AOD482, Q1M3 AOD482, Q1M4 AOD482, U1M1 VNH5019, U1M2 VNH5019, U1M3 VNH5019, U1M4 VNH5019, X1 BM10B-SRSS-TB

Commit message: Change pullup resistor to value we alr have
Parts:
- R1M1, R1M2, R1M3, R1M4, R2M1, R2M2, R2M3, R2M4: value 3.3k -> 3.24k
Changed lines of the file:
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@@
 <drawing>
 <settings>
-<setting alwaysvectorfont="no"/>
+<setting alwaysvectorfont="yes"/>
 <setting verticaltext="up"/>
 </settings>
@@
 <attribute name="NAME" x="-30.322184375" y="21.686184375" size="0.7112" layer="25" font="vector" ratio="18" rot="R225" align="bottom-center"/>
 </element>
-<element name="R1M1" library="JH" library_urn="urn:adsk.eagle:library:6027132" package="R0603" package3d_urn="urn:adsk.eagle:package:15441228/3" value="3.3k" x="-29.21" y="24.765" smashed="yes" rot="R225">
+<element name="R1M1" library="JH" library_urn="urn:adsk.eagle:library:6027132" package="R0603" package3d_urn="urn:adsk.eagle:package:15441228/3" value="3.24k" x="-29.21" y="24.765" smashed="yes" rot="R225">
 <attribute name="NAME" x="-31.592184375" y="22.956184375" size="0.7112" layer="25" font="vector" ratio="18" rot="R225" align="bottom-center"/>
 </element>
-<element name="R2M1" library="JH" library_urn="urn:adsk.eagle:library:6027132" package="R0603" package3d_urn="urn:adsk.eagle:package:15441228/3" value="3.3k" x="-35.56" y="31.115" smashed="yes" rot="R225">
+<element name="R2M1" library="JH" library_urn="urn:adsk.eagle:library:6027132" package="R0603" package3d_urn="urn:adsk.eagle:package:15441228/3" value="3.24k" x="-35.56" y="31.115" smashed="yes" rot="R225">
 <attribute name="NAME" x="-37.368815625" y="28.478815625" size="0.7112" layer="25" font="vector" ratio="18" rot="R45" align="bottom-center"/>
 </element>
@@
 <attribute name="NAME" x="8.986184375" y="41.371184375" size="0.7112" layer="25" font="vector" ratio="18" rot="R135" align="bottom-center"/>
 </element>
-<element name="R1M2" library="JH" library_urn="urn:adsk.eagle:library:6027132" package="R0603" package3d_urn="urn:adsk.eagle:package:15441228/3" value="3.3k" x="10.795" y="43.18" smashed="yes" rot="R135">
+<element name="R1M2" library="JH" library_urn="urn:adsk.eagle:library:6027132" package="R0603" package3d_urn="urn:adsk.eagle:package:15441228/3" value="3.24k" x="10.795" y="43.18" smashed="yes" rot="R135">
 <attribute name="NAME" x="8.986184375" y="45.435184375" size="0.7112" layer="25" font="vector" ratio="18" rot="R135" align="bottom-center"/>
 </element>
-<element name="R2M2" library="JH" library_urn="urn:adsk.eagle:library:6027132" package="R0603" package3d_urn="urn:adsk.eagle:package:15441228/3" value="3.3k" x="17.145" y="49.53" smashed="yes" rot="R135">
+<element name="R2M2" library="JH" library_urn="urn:adsk.eagle:library:6027132" package="R0603" package3d_urn="urn:adsk.eagle:package:15441228/3" value="3.24k" x="17.145" y="49.53" smashed="yes" rot="R135">
 <attribute name="NAME" x="15.336184375" y="51.912184375" size="0.7112" layer="25" font="vector" ratio="18" rot="R135" align="bottom-center"/>
 </element>
@@
 <attribute name="NAME" x="16.4138125" y="-52.6088125" size="0.7112" layer="25" font="vector" ratio="18" rot="R225" align="bottom-center"/>
 </element>
-<element name="R1M3" library="JH" library_urn="urn:adsk.eagle:library:6027132" package="R0603" package3d_urn="urn:adsk.eagle:package:15441228/3" value="3.3k" x="17.145" y="-49.53" smashed="yes" rot="R225">
+<element name="R1M3" library="JH" library_urn="urn:adsk.eagle:library:6027132" package="R0603" package3d_urn="urn:adsk.eagle:package:15441228/3" value="3.24k" x="17.145" y="-49.53" smashed="yes" rot="R225">
 <attribute name="NAME" x="15.1438125" y="-51.3388125" size="0.7112" layer="25" font="vector" ratio="18" rot="R225" align="bottom-center"/>
 </element>
-<element name="R2M3" library="JH" library_urn="urn:adsk.eagle:library:6027132" package="R0603" package3d_urn="urn:adsk.eagle:package:15441228/3" value="3.3k" x="10.795" y="-43.18" smashed="yes" rot="R225">
+<element name="R2M3" library="JH" library_urn="urn:adsk.eagle:library:6027132" package="R0603" package3d_urn="urn:adsk.eagle:package:15441228/3" value="3.24k" x="10.795" y="-43.18" smashed="yes" rot="R225">
 <attribute name="NAME" x="8.1588125" y="-44.3538125" size="0.7112" layer="25" font="vector" ratio="18" rot="R225" align="bottom-center"/>
 </element>
@@
 <attribute name="NAME" x="-38.8928125" y="-29.8758125" size="0.7112" layer="25" font="vector" ratio="18" rot="R135" align="bottom-center"/>
 </element>
-<element name="R1M4" library="JH" library_urn="urn:adsk.eagle:library:6027132" package="R0603" package3d_urn="urn:adsk.eagle:package:15441228/3" value="3.3k" x="-35.56" y="-31.115" smashed="yes" rot="R135">
+<element name="R1M4" library="JH" library_urn="urn:adsk.eagle:library:6027132" package="R0603" package3d_urn="urn:adsk.eagle:package:15441228/3" value="3.24k" x="-35.56" y="-31.115" smashed="yes" rot="R135">
 <attribute name="NAME" x="-37.6228125" y="-28.6058125" size="0.7112" layer="25" font="vector" ratio="18" rot="R135" align="bottom-center"/>
 </element>
-<element name="R2M4" library="JH" library_urn="urn:adsk.eagle:library:6027132" package="R0603" package3d_urn="urn:adsk.eagle:package:15441228/3" value="3.3k" x="-29.21" y="-24.765" smashed="yes" rot="R135">
+<element name="R2M4" library="JH" library_urn="urn:adsk.eagle:library:6027132" package="R0603" package3d_urn="urn:adsk.eagle:package:15441228/3" value="3.24k" x="-29.21" y="-24.765" smashed="yes" rot="R135">
 <attribute name="NAME" x="-30.3838125" y="-22.1288125" size="0.7112" layer="25" font="vector" ratio="18" rot="R135" align="bottom-center"/>
 </element>
