File: PCB2k20/Layer1.brd (EAGLE design)
At the start: 173.9 x 196 mm, 281 parts, among them J1 XT30PB-F, J10 14AWG, J11 14AWG, J13 14AWG, J14 14AWG, J15 14AWG, J16 14AWG, J17 14AWG, J18 14AWG, J19 14AWG, J20 14AWG, J21 14AWG, J3 14AWG, J4 14AWG, J5 14AWG, J6 14AWG, J7 14AWG, J8 14AWG, J9 14AWG, Q1M1 AOD482, Q1M2 AOD482, Q1M3 AOD482, Q1M4 AOD482, U1M1 VNH5019, U1M2 VNH5019, U1M3 VNH5019, U1M4 VNH5019, X1 BM10B-SRSS-TB

Commit message: BROKEN VERSION for 3d models
Parts:
- removed LIGHT, S1: (no value), SparkFun-Switches:SWITCH_SPDT_PTH_11.6X4.0MM_LOCK
- added U$30, U$31: SWITCH_SPDT_TH, JH:SWITCH_SPDT_PTH_11.6X4.0MM_LOCK
- 1D0, D1M1, D1M2, D1M3, D1M4, D2M1, D2M2, D2M3, D2M4: device SparkFun-LED:LED-0603 -> JH:LED-0603
- 1OSC: device SparkFun-Clocks:CRYSTAL-SMD-5X3.2-2PAD -> JH:CRYSTAL-SMD-5X3.2-2PAD
- 1PT1, 1PT10, 1PT11, 1PT12, 1PT13, 1PT14, 1PT15, 1PT16, 1PT17, 1PT18, 1PT19, 1PT2, 1PT20, 1PT21, 1PT22, 1PT23, 1PT24, 1PT25, 1PT26, 1PT27, 1PT28, 1PT29, 1PT3, 1PT30, 1PT31, 1PT32, 1PT33, 1PT34, 1PT35, 1PT36, 1PT37, 1PT38, 1PT4, 1PT5, 1PT6, 1PT7, 1PT8, 1PT9: value LIGHT_SENSORALS -> LIGHT_SENSOR_ALS; device SparkFun-Sensors:ALS-PT19 -> JH:ALS-PT19
- 2D1: device SparkFun-DiscreteSemi:SMA-DIODE -> JH:SMA-DIODE
- 3C3: value 100uF -> CAPACITOR_POL_10X10.5MM; device SparkFun-Capacitors:NIC_10X10.5_CAP -> JH:10X10.5_CAP
- 3D4: value 1N4728 -> DIODE-ZENER; device diode:DO41Z10 -> JH:DO41Z10
- 3Q3: device SparkFun-DiscreteSemi:TO220V -> JH:TO220V
- 3Q4: device SparkFun-DiscreteSemi:SOT23-3 -> JH:SOT23-3
- FB1, FB2: value 30Ω/1.8A -> FERRITE_BEAD; device SparkFun-Coils:0603 -> JH:R0603
- J2: device SparkFun-Connectors:1X04 -> Connectors:1X04_LOCK
- MOUSE: device SparkFun-Connectors:1X08_LOCK -> Connectors:1X08_LOCK
- Q1M1, Q1M2, Q1M3, Q1M4: device SparkFun-DiscreteSemi:DPAK -> JH:DPAK
Connections:
- net 3.3V: now also U$31.1; no longer S1.1
- net 3.3V_MCU: now also U$31.2; no longer S1.2
- net 3.3V_PROG: now also U$31.3; no longer S1.3
- net N$3: now also U$30.3; no longer LIGHT.3
- net N$36: now also U$30.2; no longer LIGHT.2
- net N$58: now also U1M1.P$19, U1M1.P$20, U1M1.P$21, U1M1.P$22, U1M1.P$23, U1M1.P$24, U1M1.P$25, U1M1.P$26, U1M1.P$27, U1M1.P$28
- net N$66: now also U1M2.P$19, U1M2.P$20, U1M2.P$21, U1M2.P$22, U1M2.P$23, U1M2.P$24, U1M2.P$25, U1M2.P$26, U1M2.P$27, U1M2.P$28
- net N$74: now also U1M3.P$19, U1M3.P$20, U1M3.P$21, U1M3.P$22, U1M3.P$23, U1M3.P$24, U1M3.P$25, U1M3.P$26, U1M3.P$27, U1M3.P$28
- net N$82: now also U1M4.P$19, U1M4.P$20, U1M4.P$21, U1M4.P$22, U1M4.P$23, U1M4.P$24, U1M4.P$25, U1M4.P$26, U1M4.P$27, U1M4.P$28
- net OUTAM1: now also U1M1.P$1, U1M1.P$2, U1M1.P$3, U1M1.P$4, U1M1.P$5, U1M1.P$6, U1M1.P$7, U1M1.P$8, U1M1.P$9
- net OUTAM2: now also U1M2.P$1, U1M2.P$2, U1M2.P$3, U1M2.P$4, U1M2.P$5, U1M2.P$6, U1M2.P$7, U1M2.P$8, U1M2.P$9
- net OUTAM3: now also U1M3.P$1, U1M3.P$2, U1M3.P$3, U1M3.P$4, U1M3.P$5, U1M3.P$6, U1M3.P$7, U1M3.P$8, U1M3.P$9
- net OUTAM4: now also U1M4.P$1, U1M4.P$2, U1M4.P$3, U1M4.P$4, U1M4.P$5, U1M4.P$6, U1M4.P$7, U1M4.P$8, U1M4.P$9
- net OUTBM1: now also U1M1.P$10, U1M1.P$11, U1M1.P$12, U1M1.P$13, U1M1.P$14, U1M1.P$15, U1M1.P$16, U1M1.P$17, U1M1.P$18
- net OUTBM2: now also U1M2.P$10, U1M2.P$11, U1M2.P$12, U1M2.P$13, U1M2.P$14, U1M2.P$15, U1M2.P$16, U1M2.P$17, U1M2.P$18
- net OUTBM3: now also U1M3.P$10, U1M3.P$11, U1M3.P$12, U1M3.P$13, U1M3.P$14, U1M3.P$15, U1M3.P$16, U1M3.P$17, U1M3.P$18
- net OUTBM4: now also U1M4.P$10, U1M4.P$11, U1M4.P$12, U1M4.P$13, U1M4.P$14, U1M4.P$15, U1M4.P$16, U1M4.P$17, U1M4.P$18
Routing:
- net 3.3V_MCU: track 68.0 -> 60.7 mm
- net N$3: track 4.61 -> 1.87 mm
- net N$36: track 5.23 -> 2.69 mm
- net 3.3V_PROG: track 18.5 -> 17.7 mm
