File: PCB2k20/RescueLS.brd (EAGLE design)
At the start: 68 x 37.5 mm, 55 parts, among them J3 JST_04-V

Commit message: update values
Parts:
- 1C9: value (none) -> 1uF
- 1R2: value 15 -> 1.25
- 1R3: value 100k -> 10k
- 1R6: value (none) -> 3k
Changed lines of the file:
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@@
 <drawing>
 <settings>
-<setting alwaysvectorfont="yes"/>
+<setting alwaysvectorfont="no"/>
 <setting verticaltext="up"/>
 </settings>
@@
 </element>
 <element name="LED1" library="JH" library_urn="urn:adsk.eagle:library:6027132" package="3528" package3d_urn="urn:adsk.eagle:package:6740529/3" value="3528LED" x="-27.94" y="3.175" smashed="yes" rot="MR270"/>
-<element name="1R2" library="JH" library_urn="urn:adsk.eagle:library:6027132" package="R0603" package3d_urn="urn:adsk.eagle:package:15441228/3" value="15" x="-10.795" y="-12.065" smashed="yes" rot="MR270">
+<element name="1R2" library="JH" library_urn="urn:adsk.eagle:library:6027132" package="R0603" package3d_urn="urn:adsk.eagle:package:15441228/3" value="1.25" x="-10.795" y="-12.065" smashed="yes" rot="MR270">
 <attribute name="NAME" x="-11.557" y="-12.065" size="0.7112" layer="26" font="vector" ratio="18" rot="MR270" align="bottom-center"/>
 <attribute name="VALUE" x="-10.033" y="-12.065" size="0.7112" layer="28" font="vector" ratio="18" rot="MR270" align="top-center"/>
@@
 <attribute name="VALUE" x="10.16" y="4.953" size="0.7112" layer="27" font="vector" ratio="18" align="top-center"/>
 </element>
-<element name="1R3" library="JH" library_urn="urn:adsk.eagle:library:6027132" package="R0603" package3d_urn="urn:adsk.eagle:package:15441228/3" value="100k" x="-9.525" y="6.985" smashed="yes" rot="R270">
+<element name="1R3" library="JH" library_urn="urn:adsk.eagle:library:6027132" package="R0603" package3d_urn="urn:adsk.eagle:package:15441228/3" value="10k" x="-9.525" y="6.985" smashed="yes" rot="R270">
 <attribute name="NAME" x="-9.525" y="9.017" size="0.7112" layer="25" font="vector" ratio="18" align="bottom-center"/>
 <attribute name="VALUE" x="-9.525" y="4.953" size="0.7112" layer="27" font="vector" ratio="18" align="top-center"/>
 </element>
-<element name="1R6" library="JH" library_urn="urn:adsk.eagle:library:6027132" package="R0603" package3d_urn="urn:adsk.eagle:package:15441228/3" value="" x="12.7" y="14.605" smashed="yes" rot="R90">
+<element name="1R6" library="JH" library_urn="urn:adsk.eagle:library:6027132" package="R0603" package3d_urn="urn:adsk.eagle:package:15441228/3" value="3k" x="12.7" y="14.605" smashed="yes" rot="R90">
 <attribute name="NAME" x="11.938" y="14.605" size="0.7112" layer="25" font="vector" ratio="18" rot="R90" align="bottom-center"/>
 <attribute name="VALUE" x="13.462" y="14.605" size="0.7112" layer="27" font="vector" ratio="18" rot="R90" align="top-center"/>
 </element>
-<element name="1C9" library="JH" library_urn="urn:adsk.eagle:library:6027132" package="C0603" package3d_urn="urn:adsk.eagle:package:15441226/3" value="" x="10.16" y="14.605" smashed="yes" rot="R270">
+<element name="1C9" library="JH" library_urn="urn:adsk.eagle:library:6027132" package="C0603" package3d_urn="urn:adsk.eagle:package:15441226/3" value="1uF" x="10.16" y="14.605" smashed="yes" rot="R270">
 <attribute name="NAME" x="9.398" y="14.605" size="0.7112" layer="25" font="vector" ratio="18" rot="R90" align="bottom-center"/>
 <attribute name="VALUE" x="9.398" y="14.605" size="0.7112" layer="27" font="vector" ratio="18" rot="R270" align="top-center"/>

Commit message: Welp I should go kms dumb mistakes time for Rescue PCB V2
Parts:
- added LED13, LED14: 3528LED, JH:3528
- added PT14, PT15: LIGHT_SENSORALS, SparkFun-Sensors:ALS-PT19
- moved 1S2 21.1 mm to (0.00, -6.35), turned to 0 degrees
- moved 1R5 19.3 mm to (1.91, -2.54), turned to 270 degrees
- moved C1 18.2 mm to (-22.0, -8.13)
- moved C20 18.2 mm to (22.0, -8.13)
- moved CS1 18.0 mm to (22.0, -3.81)
- moved CS2 18.0 mm to (-22.0, -3.81)
- moved 1R4 14.9 mm to (-2.29, -2.54), turned to 90 degrees
- moved 1R2 2.01 mm to (-12.7, -11.4), turned to 180 degrees
- moved 1D1 0.63 mm to (-2.54, -12.1)
- moved 1R1 0.63 mm to (0.00, -12.1)
- moved SWD 0.63 mm to (14.6, -5.71)
- moved 1C3 0.51 mm to (4.95, -12.1)
- flipped 1C9 to the bottom
- flipped 1R6 to the bottom
Connections:
- new net N$1: 1U2.P8, PT14.E
- new net N$11: 1U2.P7, PT15.E
- net 3.3V: no longer C1.2, C20.2, CS1.5, CS2.5
- net 3.3V_MCU: now also C1.2, C20.2, CS1.5, CS2.5
- net CS1: now also 1U1.29; no longer 1U1.11
- net GND: now also LED13.C, LED14.C
- net N$3: now also LED13.A, LED14.A
- net VCCA: now also PT14.C, PT15.C
Routing:
- net S0: track 20.7 -> 66.1 mm, vias 1 -> 4
- net S1: track 16.4 -> 59.7 mm, vias 1 -> 2
- net N$11: track 0.00 -> 42.1 mm, vias 0 -> 1
- net N$1: track 0.00 -> 40.2 mm, vias 0 -> 1
- net 3.3V_MCU: track 107.0 -> 142.6 mm
- net S2: track 23.7 -> 57.9 mm, vias 1 -> 4
- net S3: track 27.8 -> 60.3 mm, vias 1 -> 4
- net 3.3V: track 57.6 -> 32.0 mm
- net CS2: track 8.24 -> 29.0 mm
- net CS1: track 8.50 -> 22.7 mm
- net VCCA: track 110.0 -> 124.1 mm
- net RESET: track 20.5 -> 8.02 mm
- net N$3: track 89.3 -> 98.4 mm
- net LSOUT: track 44.6 -> 49.7 mm, vias 2 -> 3
- net AGND: track 61.9 -> 65.7 mm, vias 4 -> 5
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Other:
- board size 68 x 37.5 mm -> 78 x 37.5 mm
